File: dropbot-front-pannel.sch (KiCad schematic (older format))
At the start: 11 parts, among them P1 CONN_02X10, P2 CONN_02X25, P3 CONN_02X20, P4 CONN_02X25, P5 CONN_02X20, P6 CONN_02X25, P7 CONN_02X20, P8 CONN_02X10, P9 CONN_01X03

Commit message: Update documentation on schematic and add pdf output
Connections:
- net labels added: HVAC
- wire segments 10 -> 14
Other:
- note added: "+12 V power is provided by a DC power brick.\n+3.3V and +5V power are obtained using\nstep-down (buck) regulators.\n\nThe control board generates a bipolar square\nwave up to 240 Vrms (frequency = 100 Hz to\n10 kHz) with a boost converter that uses the\n+12 V source as input. It communicates\nwith the computer over USB/serial and with\nthe HV switching boards over i2c.\n\nIt also measures the ret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"
- note added: "CONTROL BOARD EDGE CONNECTOR"
- note added: "DMF DEVICE CONNECTOR PORTS\nThese connectors accept high-density discrete cables (Samtec 0.050" pitch Tiger Eye series). The cables connect\nthese outputs to another PCB that interfaces with a DMF device using spring-loaded pogo-pins. Each pin carries \na bipolar square wave signal of up to 240 Vrms (frequency = 100 Hz to 10 kHz)"
- note added: "HV SWITCHING BOARD EDGE CONNECTORS\nEach switching boards consists of an array of 40 solid-state relays controlled over i2c.\nEach output is either connected to this HVAC signal or shorted to HVGND.\nHVAC is a bipolar square wave signal of up to 240 Vrms (frequency = 100 Hz to 10 kHz)"
- note added: "J1 connects HVGND to GND (note that this\nshould normally be connected)"
- note added: "J2 must be connected to enable HV output"
- note added: "JUMPERS"
- note added: "POWER AND COMMUNICATION HEADERS\nThese headers are exposed for testing and for\ncontrol by a PC or embeded linux system."
- note added: "Reset lines for the switching\nboards can be used for\nfirmware flashing."
- note removed: "CONTROL BOARD CONNECTOR"
- note removed: "HV SWITCHING BOARD CONNECTORS"

Commit message: Update BOM
Parts:
- P1: Mfg_Part_No (none) -> HSEC8-110-01-L-DV-A
- P2, P4, P6: Mfg_Part_No (none) -> HSEC8-125-01-L-DV-A
- P3, P5, P7: Mfg_Part_No (none) -> TFML-120-01-S-D
Connections:
- wire segments 14 -> 10
Changed lines of the file:
@@
 LIBS:valves
 LIBS:wheelerlab
-LIBS:dropbot-front-pannel-cache
 EELAYER 25 0
 EELAYER END
@@
 F 2 "WheelerLab:HSEC8-110-XX-X-DV" H 1550 200 50  0001 C CNN
 F 3 "" H 1550 200 50  0000 C CNN
+F 4 "HSEC8-110-01-L-DV-A" H 1550 1400 60  0001 C CNN "Mfg_Part_No"
 	1    1550 1400
 	1    0    0    -1
@@
 +5V
 Wire Wire Line
-	1300 1550 1300 1650
-Wire Wire Line
-	1300 1650 1300 1750
+	1300 1550 1300 1750
 Text GLabel 1800 1550 2    60   Input ~ 0
 GND
@@
 F 2 "WheelerLab:HSEC8-125-XX-X-DV" H 4000 1650 50  0001 C CNN
 F 3 "" H 4000 1650 50  0000 C CNN
+F 4 "HSEC8-125-01-L-DV-A" H 4000 2400 60  0001 C CNN "Mfg_Part_No"
 	1    4000 2400
 	1    0    0    -1
@@
 F 2 "WheelerLab:TFML-120-02-S-D" H 4000 4450 50  0001 C CNN
 F 3 "" H 4000 4450 50  0000 C CNN
+F 4 "TFML-120-01-S-D" H 4000 5400 60  0001 C CNN "Mfg_Part_No"
 	1    4000 5400
 	1    0    0    1
@@
 F 2 "WheelerLab:HSEC8-125-XX-X-DV" H 5900 1650 50  0001 C CNN
 F 3 "" H 5900 1650 50  0000 C CNN
+F 4 "HSEC8-125-01-L-DV-A" H 5900 2400 60  0001 C CNN "Mfg_Part_No"
 	1    5900 2400
 	1    0    0    -1
@@
 F 2 "WheelerLab:HSEC8-125-XX-X-DV" H 7800 1650 50  0001 C CNN
 F 3 "" H 7800 1650 50  0000 C CNN
+F 4 "HSEC8-125-01-L-DV-A" H 7800 2400 60  0001 C CNN "Mfg_Part_No"
 	1    7800 2400
 	1    0    0    -1
@@
 F 2 "WheelerLab:TFML-120-02-S-D" H 5900 4450 50  0001 C CNN
 F 3 "" H 5900 4450 50  0000 C CNN
+F 4 "TFML-120-01-S-D" H 5900 5400 60  0001 C CNN "Mfg_Part_No"
 	1    5900 5400
 	1    0    0    1
@@
 F 2 "WheelerLab:TFML-120-02-S-D" H 7800 4450 50  0001 C CNN
 F 3 "" H 7800 4450 50  0000 C CNN
+F 4 "TFML-120-01-S-D" H 7800 5400 60  0001 C CNN "Mfg_Part_No"
 	1    7800 5400
 	1    0    0    1
@@
 GND
 Wire Wire Line
-	1800 1350 1800 1450
-Wire Wire Line
-	1800 1450 1800 1550
+	1800 1350 1800 1550
 Text GLabel 1800 1250 2    60   Input ~ 0
 HV_OE
@@
 +5V
 Wire Wire Line
-	1350 4950 1350 5050
-Wire Wire Line
-	1350 5050 1350 5150
+	1350 4950 1350 5150
 Text GLabel 1850 4950 2    60   Input ~ 0
 GND
@@
 Connection ~ 1350 5050
 Wire Wire Line
-	1850 4750 1850 4850
-Wire Wire Line
-	1850 4850 1850 4950
+	1850 4750 1850 4950
 Text GLabel 1850 4650 2    60   Input ~ 0
 HV_OE

Commit message: Fix BOM
Parts:
- P3: Mfg_Part_No TFML-120-01-S-D -> TFML-120-02-S-D
Changed lines of the file:
@@
 F 2 "WheelerLab:TFML-120-02-S-D" H 4000 4450 50  0001 C CNN
 F 3 "" H 4000 4450 50  0000 C CNN
-F 4 "TFML-120-01-S-D" H 4000 5400 60  0001 C CNN "Mfg_Part_No"
+F 4 "TFML-120-02-S-D" H 4000 5400 60  0001 C CNN "Mfg_Part_No"
 	1    4000 5400
 	1    0    0    1

Commit message: Fix BOM
Parts:
- P5, P7: Mfg_Part_No TFML-120-01-S-D -> TFML-120-02-S-D
Changed lines of the file:
@@
 LIBS:valves
 LIBS:wheelerlab
+LIBS:dropbot-front-pannel-cache
 EELAYER 25 0
 EELAYER END
@@
 F 2 "WheelerLab:TFML-120-02-S-D" H 5900 4450 50  0001 C CNN
 F 3 "" H 5900 4450 50  0000 C CNN
-F 4 "TFML-120-01-S-D" H 5900 5400 60  0001 C CNN "Mfg_Part_No"
+F 4 "TFML-120-02-S-D" H 5900 5400 60  0001 C CNN "Mfg_Part_No"
 	1    5900 5400
 	1    0    0    1
@@
 F 2 "WheelerLab:TFML-120-02-S-D" H 7800 4450 50  0001 C CNN
 F 3 "" H 7800 4450 50  0000 C CNN
-F 4 "TFML-120-01-S-D" H 7800 5400 60  0001 C CNN "Mfg_Part_No"
+F 4 "TFML-120-02-S-D" H 7800 5400 60  0001 C CNN "Mfg_Part_No"
 	1    7800 5400
 	1    0    0    1

Commit message: [WIP] Update PCB to use Samtec connectors
Update PCB to use Samtec connectors instead of PCB edge connections.

This is because the edge connector slots are not rated for high-voltage
(i.e., they are not rated for over 30V).
Parts:
- removed P3, P5, P7: CONN_02X20, WheelerLab:TFML-120-02-S-D, symbol CONN_02X20
- added J1, J3: TFM-120-02-X-DH, WheelerLab:TFM-120-02-X-DH, symbol TFM-120-02-X-DH
- added J2: TFM-125-02-X-DH, WheelerLab:TFM-125-02-X-DH, symbol TFM-125-02-X-DH
- JP1, JP2: symbol JUMPER -> Jumper
Changed lines of the file:
@@
 EESchema Schematic File Version 2
+LIBS:dropbot-front-pannel-rescue
 LIBS:power
 LIBS:device
@@
 Text GLabel 4250 3400 2    60   Input ~ 0
 SCL
-$Comp
-L CONN_02X25 P2
-U 1 1 5847A5CC
-P 4000 2400
-F 0 "P2" H 4000 3700 50  0000 C CNN
-F 1 "CONN_02X25" V 4000 2400 50  0000 C CNN
-F 2 "WheelerLab:HSEC8-125-XX-X-DV" H 4000 1650 50  0001 C CNN
-F 3 "" H 4000 1650 50  0000 C CNN
-F 4 "HSEC8-125-01-L-DV-A" H 4000 2400 60  0001 C CNN "Mfg_Part_No"
-	1    4000 2400
-	1    0    0    -1
-$EndComp
 Text GLabel 3750 3500 0    60   Input ~ 0
 GND
@@
 Text GLabel 3750 3300 0    60   Input ~ 0
 GND
-$Comp
-L CONN_02X20 P3
-U 1 1 5847A9FB
-P 4000 5400
-F 0 "P3" H 4000 6450 50  0000 C CNN
-F 1 "CONN_02X20" V 4000 5400 50  0000 C CNN
-F 2 "WheelerLab:TFML-120-02-S-D" H 4000 4450 50  0001 C CNN
-F 3 "" H 4000 4450 50  0000 C CNN
-F 4 "TFML-120-02-S-D" H 4000 5400 60  0001 C CNN "Mfg_Part_No"
-	1    4000 5400
-	1    0    0    1
-$EndComp
 Text GLabel 3750 6250 0    60   Input ~ 0
 HVOUT36
@@
 Text GLabel 6150 3400 2    60   Input ~ 0
 SCL
-$Comp
-L CONN_02X25 P4
-U 1 1 5847BEA4
-P 5900 2400
-F 0 "P4" H 5900 3700 50  0000 C CNN
-F 1 "CONN_02X25" V 5900 2400 50  0000 C CNN
-F 2 "WheelerLab:HSEC8-125-XX-X-DV" H 5900 1650 50  0001 C CNN
-F 3 "" H 5900 1650 50  0000 C CNN
-F 4 "HSEC8-125-01-L-DV-A" H 5900 2400 60  0001 C CNN "Mfg_Part_No"
-	1    5900 2400
-	1    0    0    -1
-$EndComp
 Text GLabel 5650 3500 0    60   Input ~ 0
 GND
@@
 Text GLabel 7550 3300 0    60   Input ~ 0
 GND
-$Comp
-L CONN_02X20 P5
-U 1 1 5847C24A
-P 5900 5400
-F 0 "P5" H 5900 6450 50  0000 C CNN
-F 1 "CONN_02X20" V 5900 5400 50  0000 C CNN
-F 2 "WheelerLab:TFML-120-02-S-D" H 5900 4450 50  0001 C CNN
-F 3 "" H 5900 4450 50  0000 C CNN
-F 4 "TFML-120-02-S-D" H 5900 5400 60  0001 C CNN "Mfg_Part_No"
-	1    5900 5400
-	1    0    0    1
-$EndComp
-$Comp
-L CONN_02X20 P7
-U 1 1 5847C290
-P 7800 5400
-F 0 "P7" H 7800 6450 50  0000 C CNN
-F 1 "CONN_02X20" V 7800 5400 50  0000 C CNN
-F 2 "WheelerLab:TFML-120-02-S-D" H 7800 4450 50  0001 C CNN
-F 3 "" H 7800 4450 50  0000 C CNN
-F 4 "TFML-120-02-S-D" H 7800 5400 60  0001 C CNN "Mfg_Part_No"
-	1    7800 5400
-	1    0    0    1
-$EndComp
 Text GLabel 5650 6250 0    60   Input ~ 0
 HVOUT76
@@
 HVGND
 $Comp
-L JUMPER JP1
+L Jumper JP1
 U 1 1 5857598B
 P 1300 6650
@@
 HVGND
 $Comp
-L JUMPER JP2
+L Jumper JP2
 U 1 1 585759FC
 P 1300 7350
@@
 Wire Bus Line
 	8700 3850 3150 3850
+$Comp
+L CONN_02X25 P4
+U 1 1 5847BEA4
+P 5900 2400
+F 0 "P4" H 5900 3700 50  0000 C CNN
+F 1 "CONN_02X25" V 5900 2400 50  0000 C CNN
+F 2 "WheelerLab:HSEC8-125-XX-X-DV" H 5900 1650 50  0001 C CNN
+F 3 "" H 5900 1650 50  0000 C CNN
+F 4 "HSEC8-125-01-L-DV-A" H 5900 2400 60  0001 C CNN "Mfg_Part_No"
+	1    5900 2400
+	1    0    0    -1
+$EndComp
+$Comp
+L CONN_02X25 P2
+U 1 1 5847A5CC
+P 4000 2400
+F 0 "P2" H 4000 3700 50  0000 C CNN
+F 1 "CONN_02X25" V 4000 2400 50  0000 C CNN
+F 2 "WheelerLab:HSEC8-125-XX-X-DV" H 4000 1650 50  0001 C CNN
+F 3 "" H 4000 1650 50  0000 C CNN
+F 4 "HSEC8-125-01-L-DV-A" H 4000 2400 60  0001 C CNN "Mfg_Part_No"
+	1    4000 2400
+	1    0    0    -1
+$EndComp
+$Comp
+L TFM-120-02-X-DH J1
+U 1 1 58B6FAE9
+P 9000 700
+F 0 "J1" H 9200 830 45  0000 L BNN
+F 1 "TFM-120-02-X-DH" H 9200 -1680 45  0000 L BNN
+F 2 "WheelerLab:TFM-120-02-X-DH" H 9030 850 20  0001 C CNN
+F 3 "" H 9000 700 60  0000 C CNN
+	1    9000 700
+	1    0    0    -1
+$EndComp
+$Comp
+L TFM-120-02-X-DH J3
+U 1 1 58B6FBB6
+P 11600 700
+F 0 "J3" H 11800 830 45  0000 L BNN
+F 1 "TFM-120-02-X-DH" H 11800 -1680 45  0000 L BNN
+F 2 "WheelerLab:TFM-120-02-X-DH" H 11630 850 20  0001 C CNN
+F 3 "" H 11600 700 60  0000 C CNN
+	1    11600 700
+	1    0    0    -1
+$EndComp
+$Comp
+L TFM-125-02-X-DH J2
+U 1 1 58B6FC4B
+P 10300 700
+F 0 "J2" H 10500 850 45  0000 L BNN
+F 1 "TFM-125-02-X-DH" H 10500 -1900 45  0000 L BNN
+F 2 "WheelerLab:TFM-125-02-X-DH" H 10330 850 20  0001 C CNN
+F 3 "" H 10300 700 60  0000 C CNN
+	1    10300 700
+	1    0    0    -1
+$EndComp
 $EndSCHEMATC

Commit message: [WIP] Update to use new Samtec connectors...
* add USB passthrough
* add 3.3V power regulator
* add reverse polarity protection on +12V power line
Parts:
- removed J1, J3: TFM-120-02-X-DH, WheelerLab:TFM-120-02-X-DH, symbol TFM-120-02-X-DH
- removed J2: TFM-125-02-X-DH, WheelerLab:TFM-125-02-X-DH, symbol TFM-125-02-X-DH
- removed P1: CONN_02X10, WheelerLab:HSEC8-110-XX-X-DV, symbol CONN_02X10
- removed P8: CONN_02X10, Pin_Headers:Pin_Header_Straight_2x10, symbol CONN_02X10
- added P1: SFM-105-02-L-D-A, WheelerLab:SFM-105-02-XXX-D-A, symbol CONN_02X05
- added P10: CONN_01X02, Connect:bornier2, symbol CONN_01X02
- added P11: USB_A, Connect:USB_A_Vertical, symbol USB_A
- added P12: USB_B, Connect:USB_B_MUSB_Straight, symbol USB_B
- added P3, P7: TFM-125-02-L-DH, WheelerLab:TFM-120-02-X-DH, symbol TFM-120-02-X-DH
- added P5: TFM-125-02-L-DH, WheelerLab:TFM-125-02-X-DH, symbol TFM-125-02-X-DH
- added Q1: IRF9388TRPBF, Power_Integrations:SO-8, symbol IRF9388TRPBF
- added U2: D24V22F3, WheelerLab:D24V22F, symbol D24V22F3
- JP1, JP2: symbol Jumper -> JUMPER
- P2, P4, P6: value CONN_02X25 -> SFM-125-02-L-D-A; footprint WheelerLab:HSEC8-125-XX-X-DV -> WheelerLab:SFM-125-02-XXX-D-A; Mfg_Part_No HSEC8-125-01-L-DV-A -> SFM-125-02-L-D-A
Connections:
- net labels added: CHASIS_GND, V_IN
- net labels removed: +5V, D+, D-, HV
- no-connect marks 0 -> 4
Other:
- note added: "+12 V power is provided by a DC power brick.\n+3.3V power is obtained using a step-down\n(buck) regulator.\n\nThe control board generates a bipolar square\nwave up to 150 Vrms (frequency = 100 Hz to\n10 kHz) with a boost converter that uses the\n+12 V source as input. It communicates\nwith the computer over USB/serial and with\nthe HV switching boards over i2c.\n\nIt also measures the return curr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"
- note added: "POWER IN\n+12V input with reverse polarity\nprotection."
- note added: "POWER REGULATORS"
- note added: "USB PASSTHROUGH"
- note removed: "+12 V power is provided by a DC power brick.\n+3.3V and +5V power are obtained using\nstep-down (buck) regulators.\n\nThe control board generates a bipolar square\nwave up to 240 Vrms (frequency = 100 Hz to\n10 kHz) with a boost converter that uses the\n+12 V source as input. It communicates\nwith the computer over USB/serial and with\nthe HV switching boards over i2c.\n\nIt also measures the ret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"
- note removed: "POWER AND COMMUNICATION HEADERS\nThese headers are exposed for testing and for\ncontrol by a PC or embeded linux system."

Commit message: [WIP] update USB parts, replace jumpers with 0805 pads
Parts:
- JP1, JP2: footprint Pin_Headers:Pin_Header_Straight_1x02 -> Resistors_SMD:R_0805
- P11: footprint Connect:USB_A_Vertical -> WheelerLab:UE27AE54100; Mfg_Part_No (none) -> UE27AE54100
- P12: footprint Connect:USB_B_MUSB_Straight -> WheelerLab:1734517-1; Mfg_Part_No (none) -> 1734517-1
Connections:
- wire segments 10 -> 19
Other:
- note added: "DMF DEVICE CONNECTOR PORTS\nThese connectors accept (Samtec 0.050" pitch TFM Tiger Eye\nseries connectors) from another PCB that interfaces with a DMF\ndevice using spring-loaded pogo-pins. Each pin carries a\nbipolar square wave signal of up to 240 Vrms\n(frequency = 100 Hz to 10 kHz)"
- note removed: "DMF DEVICE CONNECTOR PORTS\nThese connectors accept high-density discrete cables (Samtec 0.050" pitch Tiger Eye series). The cables connect\nthese outputs to another PCB that interfaces with a DMF device using spring-loaded pogo-pins. Each pin carries \na bipolar square wave signal of up to 240 Vrms (frequency = 100 Hz to 10 kHz)"
Changed lines of the file:
@@
 L JUMPER JP1
 U 1 1 5857598B
-P 1350 5250
-F 0 "JP1" H 1350 5400 50  0000 C CNN
-F 1 "JUMPER" H 1350 5170 50  0000 C CNN
-F 2 "Pin_Headers:Pin_Header_Straight_1x02" H 1350 5250 50  0001 C CNN
-F 3 "" H 1350 5250 50  0000 C CNN
-	1    1350 5250
-	1    0    0    -1
-$EndComp
-Text GLabel 1050 5250 0    60   Input ~ 0
-GND
-Text GLabel 1650 5250 2    60   Input ~ 0
+P 1450 3800
+F 0 "JP1" H 1450 3950 50  0000 C CNN
+F 1 "JUMPER" H 1450 3720 50  0000 C CNN
+F 2 "Resistors_SMD:R_0805" H 1450 3800 50  0001 C CNN
+F 3 "" H 1450 3800 50  0000 C CNN
+	1    1450 3800
+	1    0    0    -1
+$EndComp
+Text GLabel 1150 3800 0    60   Input ~ 0
+GND
+Text GLabel 1750 3800 2    60   Input ~ 0
 HVGND
 $Comp
 L JUMPER JP2
 U 1 1 585759FC
-P 1350 5750
-F 0 "JP2" H 1350 5900 50  0000 C CNN
-F 1 "JUMPER" H 1350 5670 50  0000 C CNN
-F 2 "Pin_Headers:Pin_Header_Straight_1x02" H 1350 5750 50  0001 C CNN
-F 3 "" H 1350 5750 50  0000 C CNN
-	1    1350 5750
-	1    0    0    -1
-$EndComp
-Text GLabel 1050 5750 0    60   Input ~ 0
+P 1450 4300
+F 0 "JP2" H 1450 4450 50  0000 C CNN
+F 1 "JUMPER" H 1450 4220 50  0000 C CNN
+F 2 "Resistors_SMD:R_0805" H 1450 4300 50  0001 C CNN
+F 3 "" H 1450 4300 50  0000 C CNN
+	1    1450 4300
+	1    0    0    -1
+$EndComp
+Text GLabel 1150 4300 0    60   Input ~ 0
 GND
 Text GLabel 1800 1250 2    60   Input ~ 0
 HV_OE
-Text GLabel 1650 5750 2    60   Input ~ 0
+Text GLabel 1750 4300 2    60   Input ~ 0
 HV_OE
 $Comp
 L CONN_01X03 P9
 U 1 1 5857AD4F
-P 1250 6600
-F 0 "P9" H 1250 6800 50  0000 C CNN
-F 1 "CONN_01X03" V 1350 6600 50  0000 C CNN
-F 2 "Pin_Headers:Pin_Header_Straight_1x03" H 1250 6600 50  0001 C CNN
-F 3 "" H 1250 6600 50  0000 C CNN
-	1    1250 6600
-	1    0    0    -1
-$EndComp
-Text GLabel 1050 6500 0    60   Input ~ 0
+P 1350 5150
+F 0 "P9" H 1350 5350 50  0000 C CNN
+F 1 "CONN_01X03" V 1450 5150 50  0000 C CNN
+F 2 "Pin_Headers:Pin_Header_Straight_1x03" H 1350 5150 50  0001 C CNN
+F 3 "" H 1350 5150 50  0000 C CNN
+	1    1350 5150
+	1    0    0    -1
+$EndComp
+Text GLabel 1150 5050 0    60   Input ~ 0
 RST1
-Text GLabel 1050 6600 0    60   Input ~ 0
+Text GLabel 1150 5150 0    60   Input ~ 0
 RST2
-Text GLabel 1050 6700 0    60   Input ~ 0
+Text GLabel 1150 5250 0    60   Input ~ 0
 RST3
-Text Notes 3400 8500 0    60   ~ 0
-DMF DEVICE CONNECTOR PORTS\nThese connectors accept high-density discrete cables (Samtec 0.050" pitch Tiger Eye series). The cables connect\nthese outputs to another PCB that interfaces with a DMF device using spring-loaded pogo-pins. Each pin carries \na bipolar square wave signal of up to 240 Vrms (frequency = 100 Hz to 10 kHz)
-Text Notes 750  5100 0    60   ~ 0
+Text Notes 3200 7400 0    60   ~ 0
+DMF DEVICE CONNECTOR PORTS\nThese connectors accept (Samtec 0.050" pitch TFM Tiger Eye\nseries connectors) from another PCB that interfaces with a DMF\ndevice using spring-loaded pogo-pins. Each pin carries a\nbipolar square wave signal of up to 240 Vrms\n(frequency = 100 Hz to 10 kHz)
+Text Notes 850  3650 0    60   ~ 0
 JUMPERS
-Text Notes 800  5550 0    60   ~ 0
+Text Notes 900  4100 0    60   ~ 0
 J1 connects HVGND to GND (note that this\nshould normally be connected)
-Text Notes 800  6000 0    60   ~ 0
+Text Notes 900  4550 0    60   ~ 0
 J2 must be connected to enable HV output
 Text Notes 700  3150 0    60   ~ 0
 +12 V power is provided by a DC power brick.\n+3.3V power is obtained using a step-down\n(buck) regulator.\n\nThe control board generates a bipolar square\nwave up to 150 Vrms (frequency = 100 Hz to\n10 kHz) with a boost converter that uses the\n+12 V source as input. It communicates\nwith the computer over USB/serial and with\nthe HV switching boards over i2c.\n\nIt also measures the return current from the\ndevice (CUR_SENSE).
-Text Notes 1450 6650 0    60   ~ 0
+Text Notes 1550 5200 0    60   ~ 0
 Reset lines for the switching\nboards can be used for\nfirmware flashing.
 $Comp
@@
 F 0 "P11" H 9600 850 50  0000 C CNN
 F 1 "USB_A" H 9350 1250 50  0000 C CNN
-F 2 "Connect:USB_A_Vertical" V 9350 950 50  0001 C CNN
+F 2 "WheelerLab:UE27AE54100" V 9350 950 50  0001 C CNN
 F 3 "" V 9350 950 50  0000 C CNN
+F 4 "UE27AE54100" H 9400 1050 60  0001 C CNN "Mfg_Part_No"
 	1    9400 1050
 	1    0    0    -1
@@
 F 0 "P12" H 9600 1450 50  0000 C CNN
 F 1 "USB_B" H 9350 1850 50  0000 C CNN
-F 2 "Connect:USB_B_MUSB_Straight" V 9350 1550 50  0001 C CNN
+F 2 "WheelerLab:1734517-1" V 9350 1550 50  0001 C CNN
 F 3 "" V 9350 1550 50  0000 C CNN
+F 4 "1734517-1" H 9400 1650 60  0001 C CNN "Mfg_Part_No"
 	1    9400 1650
 	1    0    0    -1
@@
 	8700 600  3150 600
 Wire Bus Line
-	3150 3800 3150 6950
+	3150 3800 3150 7500
 Wire Bus Line
 	8700 6650 8700 3800
@@
 $EndComp
 Wire Bus Line
-	3150 6950 6250 6950
-Wire Bus Line
-	6250 6950 6250 6650
+	3150 7500 6250 7500
+Wire Bus Line
+	6250 7500 6250 6650
 Wire Bus Line
 	6250 6650 8700 6650
+Wire Wire Line
+	3750 6150 3750 6250
+Wire Wire Line
+	3750 6250 4450 6250
+Wire Wire Line
+	4450 6250 4450 6150
+Wire Wire Line
+	5450 6650 5450 6750
+Wire Wire Line
+	5450 6750 6150 6750
+Wire Wire Line
+	6150 6750 6150 6650
+Wire Wire Line
+	7200 6150 7200 6250
+Wire Wire Line
+	7900 6150 7900 6250
+Wire Wire Line
+	7900 6250 7200 6250
 $EndSCHEMATC

Commit message: [WIP] Add EMI suppression, ESD protection
Parts:
- added C1, C2, C3, C4: 0.1uF, Capacitors_SMD:C_0805, symbol C_Small
- added D1: WE-TVS_824015, WheelerLab:wurth-WE-TVS_SOT23-6L, symbol WE-TVS_824015
- added FB1, FB2: 600 Ohm@100MHz, Resistors_SMD:R_0805, symbol FERRITE
- added L1: 90 Ohm@100MHz, WheelerLab:wurth-WE-CNSW_0805, symbol CM_CHOKE
- added L2: 1.8mH, WheelerLab:RN242-X-02-XXX, symbol CM_CHOKE
- added P13, P14, P15, P8: CONN_01X01, Connect:1pin, symbol CONN_01X01
Connections:
- net labels added: +12V_SUPPLY
- net labels removed: V_IN
- wire segments 19 -> 78
- no-connect marks 4 -> 2
Other:
- note added: "3.3V POWER REGULATOR"
- note added: "MOUNTING HOLES"
- note added: "POWER IN\n+12V input with reverse polarity protection and\nEMI filter."
- note added: "USB PASSTHROUGH\nIncludes ESD protection and\nEMI suppression (See Wurth\nElectronics App Note ANP002C)."
- note removed: "POWER IN\n+12V input with reverse polarity\nprotection."
- note removed: "POWER REGULATORS"
- note removed: "USB PASSTHROUGH"
- moved on the sheet: Q1, U2
