File: dropbot-front-pannel.sch (KiCad schematic (older format))
At the start: 28 parts, among them P1 SFM-105-02-L-D-A, P10 CONN_01X02, P11 USB_A, P12 USB_B, P13 CONN_01X01, P14 CONN_01X01, P15 CONN_01X01, P2 SFM-125-02-L-D-A, P3 TFM-125-02-L-DH, P4 SFM-125-02-L-D-A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

Commit message: [WIP] route HV outputs
Connections:
- wire segments 78 -> 58

Commit message: [WIP] swap order of switching boards
Parts:
- renumbered P6 to P2, P7 to P3, P2 to P6, P3 to P7
Changed lines of the file:
@@
 SCL
 $Comp
-L CONN_02X25 P2
+L CONN_02X25 P6
 U 1 1 5847A5CC
 P 4000 2400
-F 0 "P2" H 4000 3700 50  0000 C CNN
+F 0 "P6" H 4000 3700 50  0000 C CNN
 F 1 "SFM-125-02-L-D-A" V 4000 2400 50  0000 C CNN
 F 2 "WheelerLab:SFM-125-02-XXX-D-A" H 4000 1650 50  0001 C CNN
@@
 HVOUT81
 $Comp
-L CONN_02X25 P6
+L CONN_02X25 P2
 U 1 1 5847C137
 P 7800 2400
-F 0 "P6" H 7800 3700 50  0000 C CNN
+F 0 "P2" H 7800 3700 50  0000 C CNN
 F 1 "SFM-125-02-L-D-A" V 7800 2400 50  0000 C CNN
 F 2 "WheelerLab:SFM-125-02-XXX-D-A" H 7800 1650 50  0001 C CNN
@@
 GND
 $Comp
-L TFM-120-02-X-DH P3
+L TFM-120-02-X-DH P7
 U 1 1 58B86F28
 P 3750 4050
-F 0 "P3" H 3950 4180 45  0000 L BNN
+F 0 "P7" H 3950 4180 45  0000 L BNN
 F 1 "TFM-125-02-L-DH" V 4150 2750 45  0000 L BNN
 F 2 "WheelerLab:TFM-120-02-X-DH" H 3780 4200 20  0001 C CNN
@@
 $EndComp
 $Comp
-L TFM-120-02-X-DH P7
+L TFM-120-02-X-DH P3
 U 1 1 58B876C3
 P 7200 4050
-F 0 "P7" H 7400 4180 45  0000 L BNN
+F 0 "P3" H 7400 4180 45  0000 L BNN
 F 1 "TFM-125-02-L-DH" V 7600 2850 45  0000 L BNN
 F 2 "WheelerLab:TFM-120-02-X-DH" H 7230 4200 20  0001 C CNN

Commit message: [WIP] route power, ground planes
Connections:
- wire segments 58 -> 78
Changed lines of the file:
@@
 	1    0    0    -1
 $EndComp
-Text GLabel 5450 4250 0    60   Input ~ 0
+Text GLabel 5450 4750 0    60   Input ~ 0
 HVOUT75
-Text GLabel 5450 4150 0    60   Input ~ 0
+Text GLabel 5450 4650 0    60   Input ~ 0
 HVOUT77
-Text GLabel 5450 4050 0    60   Input ~ 0
+Text GLabel 5450 4550 0    60   Input ~ 0
 HVOUT79
-Text GLabel 5450 4350 0    60   Input ~ 0
+Text GLabel 5450 4850 0    60   Input ~ 0
 HVOUT73
+Text GLabel 5450 5650 0    60   Input ~ 0
+HVOUT57
+Text GLabel 5450 5550 0    60   Input ~ 0
+HVOUT59
+Text GLabel 5450 5350 0    60   Input ~ 0
+HVOUT63
+Text GLabel 5450 5450 0    60   Input ~ 0
+HVOUT61
+Text GLabel 5450 5050 0    60   Input ~ 0
+HVOUT69
+Text GLabel 5450 4950 0    60   Input ~ 0
+HVOUT71
 Text GLabel 5450 5150 0    60   Input ~ 0
-HVOUT57
-Text GLabel 5450 5050 0    60   Input ~ 0
-HVOUT59
-Text GLabel 5450 4850 0    60   Input ~ 0
-HVOUT63
-Text GLabel 5450 4950 0    60   Input ~ 0
-HVOUT61
-Text GLabel 5450 4550 0    60   Input ~ 0
-HVOUT69
-Text GLabel 5450 4450 0    60   Input ~ 0
-HVOUT71
-Text GLabel 5450 4650 0    60   Input ~ 0
 HVOUT67
-Text GLabel 5450 4750 0    60   Input ~ 0
+Text GLabel 5450 5250 0    60   Input ~ 0
 HVOUT65
-Text GLabel 5450 5550 0    60   Input ~ 0
+Text GLabel 5450 6050 0    60   Input ~ 0
 HVOUT49
-Text GLabel 5450 5450 0    60   Input ~ 0
+Text GLabel 5450 5950 0    60   Input ~ 0
 HVOUT51
-Text GLabel 5450 5250 0    60   Input ~ 0
+Text GLabel 5450 5750 0    60   Input ~ 0
 HVOUT55
-Text GLabel 5450 5350 0    60   Input ~ 0
+Text GLabel 5450 5850 0    60   Input ~ 0
 HVOUT53
-Text GLabel 5450 5750 0    60   Input ~ 0
+Text GLabel 5450 6250 0    60   Input ~ 0
 HVOUT45
-Text GLabel 5450 5650 0    60   Input ~ 0
+Text GLabel 5450 6150 0    60   Input ~ 0
 HVOUT47
-Text GLabel 5450 5850 0    60   Input ~ 0
+Text GLabel 5450 6350 0    60   Input ~ 0
 HVOUT43
-Text GLabel 5450 5950 0    60   Input ~ 0
+Text GLabel 5450 6450 0    60   Input ~ 0
 HVOUT41
 Text GLabel 7900 4150 2    60   Input ~ 0
@@
 	1    0    0    -1
 $EndComp
-Text GLabel 6150 4150 2    60   Input ~ 0
+Text GLabel 6150 4650 2    60   Input ~ 0
 HVOUT76
-Text GLabel 6150 4050 2    60   Input ~ 0
+Text GLabel 6150 4550 2    60   Input ~ 0
 HVOUT78
+Text GLabel 6150 6450 2    60   Input ~ 0
+HVOUT40
+Text GLabel 6150 4750 2    60   Input ~ 0
+HVOUT74
+Text GLabel 6150 5550 2    60   Input ~ 0
+HVOUT58
+Text GLabel 6150 5450 2    60   Input ~ 0
+HVOUT60
+Text GLabel 6150 5250 2    60   Input ~ 0
+HVOUT64
+Text GLabel 6150 5350 2    60   Input ~ 0
+HVOUT62
+Text GLabel 6150 4950 2    60   Input ~ 0
+HVOUT70
+Text GLabel 6150 4850 2    60   Input ~ 0
+HVOUT72
+Text GLabel 6150 5050 2    60   Input ~ 0
+HVOUT68
+Text GLabel 6150 5150 2    60   Input ~ 0
+HVOUT66
 Text GLabel 6150 5950 2    60   Input ~ 0
-HVOUT40
-Text GLabel 6150 4250 2    60   Input ~ 0
-HVOUT74
-Text GLabel 6150 5050 2    60   Input ~ 0
-HVOUT58
-Text GLabel 6150 4950 2    60   Input ~ 0
-HVOUT60
-Text GLabel 6150 4750 2    60   Input ~ 0
-HVOUT64
-Text GLabel 6150 4850 2    60   Input ~ 0
-HVOUT62
-Text GLabel 6150 4450 2    60   Input ~ 0
-HVOUT70
-Text GLabel 6150 4350 2    60   Input ~ 0
-HVOUT72
-Text GLabel 6150 4550 2    60   Input ~ 0
-HVOUT68
-Text GLabel 6150 4650 2    60   Input ~ 0
-HVOUT66
-Text GLabel 6150 5450 2    60   Input ~ 0
 HVOUT50
-Text GLabel 6150 5350 2    60   Input ~ 0
+Text GLabel 6150 5850 2    60   Input ~ 0
 HVOUT52
-Text GLabel 6150 5150 2    60   Input ~ 0
+Text GLabel 6150 5650 2    60   Input ~ 0
 HVOUT56
-Text GLabel 6150 5250 2    60   Input ~ 0
+Text GLabel 6150 5750 2    60   Input ~ 0
 HVOUT54
-Text GLabel 6150 5650 2    60   Input ~ 0
+Text GLabel 6150 6150 2    60   Input ~ 0
 HVOUT46
-Text GLabel 6150 5550 2    60   Input ~ 0
+Text GLabel 6150 6050 2    60   Input ~ 0
 HVOUT48
-Text GLabel 6150 5750 2    60   Input ~ 0
+Text GLabel 6150 6250 2    60   Input ~ 0
 HVOUT44
-Text GLabel 6150 5850 2    60   Input ~ 0
+Text GLabel 6150 6350 2    60   Input ~ 0
 HVOUT42
 $Comp
@@
 $EndComp
 Wire Bus Line
-	550  2800 3050 2800
-Wire Bus Line
-	3050 2800 3050 600
+	550  2750 3050 2750
+Wire Bus Line
+	3050 2750 3050 600
 Wire Bus Line
 	3050 600  550  600
 Wire Bus Line
-	550  600  550  2800
+	550  600  550  2750
 Wire Bus Line
 	3150 600  3150 3700
@@
 	550  4950 550  5950
 Wire Bus Line
-	8850 600  8850 3550
-Wire Bus Line
-	8850 3550 10450 3550
+	8800 600  8800 3550
+Wire Bus Line
+	8800 3550 10450 3550
 Wire Bus Line
 	10450 3550 10450 600
 Wire Bus Line
-	10450 600  8850 600
+	10450 600  8800 600
 Wire Bus Line
 	550  2850 3050 2850
 Wire Bus Line
-	3050 2850 3050 4900
-Wire Bus Line
-	550  4900 550  2850
+	3050 2850 3050 4850
+Wire Bus Line
+	550  4850 550  2850
 Wire Wire Line
 	950  3450 950  3250
 Wire Wire Line
-	1350 3250 1350 3650
+	1350 3250 1350 3450
+Wire Wire Line
+	1350 3450 1350 3550
+Wire Wire Line
+	1350 3550 1350 3650
 Connection ~ 1350 3450
 Connection ~ 1350 3550
 Wire Wire Line
-	1950 3450 1950 3750
+	1950 3450 1950 3550
+Wire Wire Line
+	1950 3550 1950 3650
+Wire Wire Line
+	1950 3650 1950 3750
 Connection ~ 1950 3650
 Connection ~ 1950 3550
@@
 	6250 6650 8700 6650
 Wire Wire Line
-	3750 6150 3750 6250
-Wire Wire Line
-	3750 6250 4450 6250
-Wire Wire Line
-	4450 6250 4450 6150
-Wire Wire Line
 	5450 6650 5450 6750
 Wire Wire Line
@@
 	9300 1850 9200 1850
 Wire Wire Line
-	9200 1650 9200 2550
+	9200 1650 9200 1850
+Wire Wire Line
+	9200 1850 9200 2250
+Wire Wire Line
+	9200 2250 9200 2550
 Wire Wire Line
 	9200 2250 9300 2250
 Connection ~ 9200 1850
 Wire Wire Line
-	10000 1650 10000 2550
+	10000 1650 10000 1850
+Wire Wire Line
+	10000 1850 10000 2250
+Wire Wire Line
+	10000 2250 10000 2550
 Wire Wire Line
 	10000 2250 9900 2250
@@
 	9750 1600 9950 1600
 Wire Wire Line
-	9950 1600 9950 3400
+	9950 1600 9950 2050
+Wire Wire Line
+	9950 2050 9950 3400
 Wire Wire Line
 	9950 2050 9900 2050
@@
 	950  3250 1350 3250
 Wire Wire Line
-	1950 3450 2200 3450
+	1950 3450 2050 3450
+Wire Wire Line
+	2050 3450 2200 3450
 Wire Wire Line
 	2200 3450 2200 3500
 Wire Wire Line
-	800  3950 2700 3950
+	800  3950 950  3950
+Wire Wire Line
+	950  3950 1350 3950
+Wire Wire Line
+	1350 3950 2050 3950
+Wire Wire Line
+	2050 3950 2200 3950
+Wire Wire Line
+	2200 3950 2450 3950
+Wire Wire Line
+	2450 3950 2700 3950
 Wire Wire Line
 	2200 3950 2200 3600
@@
 $EndComp
 Wire Bus Line
-	3050 4900 550  4900
+	3050 4850 550  4850
 Wire Wire Line
 	2400 3500 2700 3500
@@
 	2450 3650 2450 3600
 Wire Wire Line
-	2400 3600 2750 3600
+	2400 3600 2450 3600
+Wire Wire Line
+	2450 3600 2750 3600
 Connection ~ 2450 3600
 Wire Wire Line
@@
 $EndComp
 Wire Wire Line
-	9000 1600 9000 2300
+	9000 1600 9000 2050
+Wire Wire Line
+	9000 2050 9000 2300
 Wire Wire Line
 	9000 1600 9450 1600
@@
 $EndComp
 Wire Wire Line
-	9000 2600 9000 2800
+	9000 2600 9000 2700
+Wire Wire Line
+	9000 2700 9000 2800
 $Comp
 L C_Small C4
@@
 CHASIS_GND
 Wire Wire Line
-	1050 4400 1050 4700
+	1050 4400 1050 4500
+Wire Wire Line
+	1050 4500 1050 4600
+Wire Wire Line
+	1050 4600 1050 4700
 Connection ~ 1050 4500
 Connection ~ 1050 4600
@@
 Text Notes 650  4300 0    60   ~ 0
 MOUNTING HOLES
+Wire Wire Line
+	4450 6250 4450 6150
+Wire Wire Line
+	3750 6150 3750 6250
+Wire Wire Line
+	3750 6250 4450 6250
+Text GLabel 3750 6250 0    60   Input ~ 0
+GND
+Text GLabel 5450 6750 0    60   Input ~ 0
+GND
+Text GLabel 7200 6250 0    60   Input ~ 0
+GND
 $EndSCHEMATC

Commit message: Finish routing all nets, move components to front of board
Connections:
- net labels added: CH-X1, CH-X2, D+, D-
Other:
- note added: "DMF DEVICE CONNECTOR PORTS\nThese connectors accept (Samtec 0.050" pitch TFM Tiger Eye\nseries connectors) from another PCB that interfaces with a DMF\ndevice using spring-loaded pogo-pins. Each pin carries a\nbipolar square wave signal of up to 150 Vrms\n(frequency = 100 Hz to 10 kHz)"
- note added: "HV SWITCHING BOARD EDGE CONNECTORS\nEach switching boards consists of an array of 40 solid-state relays controlled over i2c.\nEach output is either connected to this HVAC signal or shorted to HVGND.\nHVAC is a bipolar square wave signal of up to 150 Vrms (frequency = 100 Hz to 10 kHz)"
- note removed: "DMF DEVICE CONNECTOR PORTS\nThese connectors accept (Samtec 0.050" pitch TFM Tiger Eye\nseries connectors) from another PCB that interfaces with a DMF\ndevice using spring-loaded pogo-pins. Each pin carries a\nbipolar square wave signal of up to 240 Vrms\n(frequency = 100 Hz to 10 kHz)"
- note removed: "HV SWITCHING BOARD EDGE CONNECTORS\nEach switching boards consists of an array of 40 solid-state relays controlled over i2c.\nEach output is either connected to this HVAC signal or shorted to HVGND.\nHVAC is a bipolar square wave signal of up to 240 Vrms (frequency = 100 Hz to 10 kHz)"
- moved on the sheet: P3, P5, P7

Commit message: Fix control board connector to match v3.1
Connections:
- wire segments 78 -> 58
Changed lines of the file:
@@
 Text GLabel 1300 1050 0    60   Input ~ 0
 +3.3V
+Text GLabel 1300 1350 0    60   Input ~ 0
+HVAC
 Text GLabel 1800 1350 2    60   Input ~ 0
-HVAC
-Text GLabel 1300 1350 0    60   Input ~ 0
 +12V
 Text GLabel 3750 1900 0    60   Input ~ 0
@@
 Text GLabel 950  7300 0    60   Input ~ 0
 GND
-Text GLabel 1800 1250 2    60   Input ~ 0
+Text GLabel 1800 1150 2    60   Input ~ 0
 HV_OE
 Text GLabel 1550 7300 2    60   Input ~ 0
@@
 	1    0    0    -1
 $EndComp
+Text GLabel 1800 1250 2    60   Input ~ 0
++12V
 Text GLabel 1300 1250 0    60   Input ~ 0
-+12V
-Text GLabel 1800 1150 2    60   Input ~ 0
 GND
 $Comp
@@
 	950  3450 950  3250
 Wire Wire Line
-	1350 3250 1350 3450
-Wire Wire Line
-	1350 3450 1350 3550
-Wire Wire Line
-	1350 3550 1350 3650
+	1350 3250 1350 3650
 Connection ~ 1350 3450
 Connection ~ 1350 3550
 Wire Wire Line
-	1950 3450 1950 3550
-Wire Wire Line
-	1950 3550 1950 3650
-Wire Wire Line
-	1950 3650 1950 3750
+	1950 3450 1950 3750
 Connection ~ 1950 3650
 Connection ~ 1950 3550
@@
 	9300 1850 9200 1850
 Wire Wire Line
-	9200 1650 9200 1850
-Wire Wire Line
-	9200 1850 9200 2250
-Wire Wire Line
-	9200 2250 9200 2550
+	9200 1650 9200 2550
 Wire Wire Line
 	9200 2250 9300 2250
 Connection ~ 9200 1850
 Wire Wire Line
-	10000 1650 10000 1850
-Wire Wire Line
-	10000 1850 10000 2250
-Wire Wire Line
-	10000 2250 10000 2550
+	10000 1650 10000 2550
 Wire Wire Line
 	10000 2250 9900 2250
@@
 	9750 1600 9950 1600
 Wire Wire Line
-	9950 1600 9950 2050
-Wire Wire Line
-	9950 2050 9950 3400
+	9950 1600 9950 3400
 Wire Wire Line
 	9950 2050 9900 2050
@@
 	950  3250 1350 3250
 Wire Wire Line
-	1950 3450 2050 3450
-Wire Wire Line
-	2050 3450 2200 3450
+	1950 3450 2200 3450
 Wire Wire Line
 	2200 3450 2200 3500
 Wire Wire Line
-	800  3950 950  3950
-Wire Wire Line
-	950  3950 1350 3950
-Wire Wire Line
-	1350 3950 2050 3950
-Wire Wire Line
-	2050 3950 2200 3950
-Wire Wire Line
-	2200 3950 2450 3950
-Wire Wire Line
-	2450 3950 2700 3950
+	800  3950 2700 3950
 Wire Wire Line
 	2200 3950 2200 3600
@@
 	2450 3650 2450 3600
 Wire Wire Line
-	2400 3600 2450 3600
-Wire Wire Line
-	2450 3600 2750 3600
+	2400 3600 2750 3600
 Connection ~ 2450 3600
 Wire Wire Line
@@
 $EndComp
 Wire Wire Line
-	9000 1600 9000 2050
-Wire Wire Line
-	9000 2050 9000 2300
+	9000 1600 9000 2300
 Wire Wire Line
 	9000 1600 9450 1600
@@
 $EndComp
 Wire Wire Line
-	9000 2600 9000 2700
-Wire Wire Line
-	9000 2700 9000 2800
+	9000 2600 9000 2800
 $Comp
 L C_Small C4
@@
 CHASIS_GND
 Wire Wire Line
-	1050 4400 1050 4500
-Wire Wire Line
-	1050 4500 1050 4600
-Wire Wire Line
-	1050 4600 1050 4700
+	1050 4400 1050 4700
 Connection ~ 1050 4500
 Connection ~ 1050 4600
@@
 Text GLabel 5500 4050 0    60   Input ~ 0
 CH-X2
-Text GLabel 5450 4150 0    60   Input ~ 0
+Text GLabel 5500 4150 0    60   Input ~ 0
 CUR_SENSE
 Text GLabel 5500 4250 0    60   Input ~ 0

Commit message: Remove usb passthrough, fix SMT connector...
* remove usb passthrough
* fix SMT connector footprints (missing holes)
* remove USB passthrough (now on control board)
* move power connector to top of board
* increase height of cutouts in bottom corners
Parts:
- removed C4: 0.1uF, Capacitors_SMD:C_0805, symbol C_Small
- removed D1: WE-TVS_824015, WheelerLab:wurth-WE-TVS_SOT23-6L, symbol WE-TVS_824015
- removed FB1, FB2: 600 Ohm@100MHz, Resistors_SMD:R_0805, symbol FERRITE
- removed L1: 90 Ohm@100MHz, WheelerLab:wurth-WE-CNSW_0805, symbol CM_CHOKE
- removed P11: USB_A, WheelerLab:UE27AE54100, symbol USB_A
- removed P12: USB_B, WheelerLab:1734517-1, symbol USB_B
- C1, C2, C3: Mfg_Part_No (none) -> CL21B104KBCNNNC
- JP1: Mfg_Part_No (none) -> RC0805JR-070RL
- P10: Mfg_Part_No (none) -> ED2609-ND
- Q1: Mfg_Part_No (none) -> IRF9388TRPBF
Connections:
- net labels removed: D+, D-
- wire segments 58 -> 28
Other:
- note removed: "USB PASSTHROUGH\nIncludes ESD protection and\nEMI suppression (See Wurth\nElectronics App Note ANP002C)."
Changed lines of the file:
@@
 Sheet 1 1
 Title "DropBot front pannel"
-Date "2017-03-08"
-Rev "0.2"
+Date "2017-03-21"
+Rev "3.0"
 Comp "Sci-Bots Inc."
 Comment1 ""
@@
 F 2 "Resistors_SMD:R_0805" H 1250 6800 50  0001 C CNN
 F 3 "" H 1250 6800 50  0000 C CNN
+F 4 "RC0805JR-070RL" H 1250 6800 60  0001 C CNN "Mfg_Part_No"
 	1    1250 6800
 	1    0    0    -1
@@
 F 2 "Connect:bornier2" H 1150 3500 50  0001 C CNN
 F 3 "" H 1150 3500 50  0000 C CNN
+F 4 "ED2609-ND" H 1150 3500 60  0001 C CNN "Mfg_Part_No"
 	1    1150 3500
 	1    0    0    -1
@@
 Text Notes 700  5100 0    60   ~ 0
 3.3V POWER REGULATOR
-$Comp
-L USB_A P11
-U 1 1 58AEE5D3
-P 9650 3100
-F 0 "P11" H 9850 2900 50  0000 C CNN
-F 1 "USB_A" H 9600 3300 50  0000 C CNN
-F 2 "WheelerLab:UE27AE54100" V 9600 3000 50  0001 C CNN
-F 3 "" V 9600 3000 50  0000 C CNN
-F 4 "UE27AE54100" H 9650 3100 60  0001 C CNN "Mfg_Part_No"
-	1    9650 3100
-	1    0    0    -1
-$EndComp
-$Comp
-L USB_B P12
-U 1 1 58AEE77B
-P 9650 1300
-F 0 "P12" H 9850 1100 50  0000 C CNN
-F 1 "USB_B" H 9600 1500 50  0000 C CNN
-F 2 "WheelerLab:1734517-1" V 9600 1200 50  0001 C CNN
-F 3 "" V 9600 1200 50  0000 C CNN
-F 4 "1734517-1" H 9650 1300 60  0001 C CNN "Mfg_Part_No"
-	1    9650 1300
-	1    0    0    -1
-$EndComp
-Text GLabel 9950 3400 2    60   Input ~ 0
-GND
-Text Notes 8900 1000 0    60   ~ 0
-USB PASSTHROUGH\nIncludes ESD protection and\nEMI suppression (See Wurth\nElectronics App Note ANP002C).
 Text Notes 600  3150 0    60   ~ 0
 POWER IN\n+12V input with reverse polarity protection and\nEMI filter.
@@
 F 2 "Power_Integrations:SO-8" H 1650 4100 50  0001 C CIN
 F 3 "" V 1650 3650 50  0000 L CNN
+F 4 "IRF9388TRPBF" H 1650 3650 60  0001 C CNN "Mfg_Part_No"
 	1    1650 3650
 	1    0    0    -1
@@
 Text GLabel 2000 5400 2    60   Input ~ 0
 GND
-Text GLabel 10150 1200 3    60   Input ~ 0
-CHASIS_GND
 $Comp
 L CONN_02X05 P1
@@
 	1    0    0    -1
 $EndComp
-$Comp
-L WE-TVS_824015 D1
-U 1 1 58BAFF99
-P 9600 2050
-F 0 "D1" V 9250 2000 45  0000 L BNN
-F 1 "WE-TVS_824015" V 10065 1850 45  0000 L BNN
-F 2 "WheelerLab:wurth-WE-TVS_SOT23-6L" H 9630 2200 20  0001 C CNN
-F 3 "" H 9600 2050 60  0000 C CNN
-F 4 "824015" H 9600 2050 60  0001 C CNN "Mfg_Part_No"
-	1    9600 2050
-	0    -1   1    0
-$EndComp
-$Comp
-L CM_CHOKE L1
-U 1 1 58BBE1AE
-P 9600 2700
-F 0 "L1" H 9450 2750 50  0000 L CNN
-F 1 "90 Ohm@100MHz" H 8850 2650 50  0000 L CNN
-F 2 "WheelerLab:wurth-WE-CNSW_0805" H 9650 2700 50  0001 C CNN
-F 3 "" H 9650 2700 50  0000 C CNN
-F 4 "744231091" H 9600 2700 60  0001 C CNN "Mfg_Part_No"
-	1    9600 2700
-	-1   0    0    -1
-$EndComp
 Wire Bus Line
 	550  2750 3050 2750
@@
 Wire Bus Line
 	550  5900 550  7700
-Wire Bus Line
-	8750 600  8750 3700
-Wire Bus Line
-	8750 3700 10400 3700
-Wire Bus Line
-	10400 3700 10400 600
-Wire Bus Line
-	10400 600  8750 600
 Wire Bus Line
 	550  2850 3050 2850
@@
 Wire Wire Line
 	8100 6250 7400 6250
-Wire Wire Line
-	9550 1650 9550 1600
-Wire Wire Line
-	9200 1650 9550 1650
-Wire Wire Line
-	9650 1600 9650 1650
-Wire Wire Line
-	9650 1650 10000 1650
-Wire Wire Line
-	9300 1850 9200 1850
-Wire Wire Line
-	9200 1650 9200 2550
-Wire Wire Line
-	9200 2250 9300 2250
-Connection ~ 9200 1850
-Wire Wire Line
-	10000 1650 10000 2550
-Wire Wire Line
-	10000 2250 9900 2250
-Wire Wire Line
-	9900 1850 10000 1850
-Connection ~ 10000 1850
-Connection ~ 9200 2250
-Connection ~ 10000 2250
-Wire Wire Line
-	9750 1600 9950 1600
-Wire Wire Line
-	9950 1600 9950 3400
-Wire Wire Line
-	9950 2050 9900 2050
-Wire Wire Line
-	9200 2550 9550 2550
-Wire Wire Line
-	10000 2550 9650 2550
-Wire Wire Line
-	9550 2800 9550 3400
-Wire Wire Line
-	9650 3400 9650 2800
-Wire Wire Line
-	9550 2550 9550 2600
-Wire Wire Line
-	9650 2550 9650 2600
 $Comp
 L CM_CHOKE L2
@@
 F 2 "Capacitors_SMD:C_0805" H 2050 3600 50  0001 C CNN
 F 3 "" H 2050 3600 50  0000 C CNN
+F 4 "CL21B104KBCNNNC" H 2050 3600 60  0001 C CNN "Mfg_Part_No"
 	1    2050 3600
 	1    0    0    -1
@@
 F 2 "Capacitors_SMD:C_0805" H 2450 3750 50  0001 C CNN
 F 3 "" H 2450 3750 50  0000 C CNN
+F 4 "CL21B104KBCNNNC" H 2450 3750 60  0001 C CNN "Mfg_Part_No"
 	1    2450 3750
 	1    0    0    -1
@@
 F 2 "Capacitors_SMD:C_0805" H 2700 3750 50  0001 C CNN
 F 3 "" H 2700 3750 50  0000 C CNN
+F 4 "CL21B104KBCNNNC" H 2700 3750 60  0001 C CNN "Mfg_Part_No"
 	1    2700 3750
 	1    0    0    -1
@@
 	2400 3600 2750 3600
 Connection ~ 2450 3600
-Wire Wire Line
-	9950 1200 10150 1200
-$Comp
-L FERRITE FB1
-U 1 1 58BE3979
-P 9000 2450
-F 0 "FB1" H 8875 2625 50  0000 L CNN
-F 1 "600 Ohm@100MHz" H 8450 2350 50  0000 L CNN
-F 2 "Resistors_SMD:R_0805" H 9000 2350 60  0001 C CNN
-F 3 "" H 9000 2350 60  0000 C CNN
-F 4 "742792040" H 9000 2450 60  0001 C CNN "Mfg_Part_No"
-	1    9000 2450
-	0    1    1    0
-$EndComp
-Wire Wire Line
-	9000 1600 9000 2300
-Wire Wire Line
-	9000 1600 9450 1600
-Wire Wire Line
-	9000 3400 9450 3400
-$Comp
-L FERRITE FB2
-U 1 1 58BE422E
-P 9000 2950
-F 0 "FB2" H 8875 3125 50  0000 L CNN
-F 1 "600 Ohm@100MHz" H 8750 2850 50  0000 L CNN
-F 2 "Resistors_SMD:R_0805" H 9000 2850 60  0001 C CNN
-F 3 "" H 9000 2850 60  0000 C CNN
-F 4 "742792040" H 9000 2950 60  0001 C CNN "Mfg_Part_No"
-	1    9000 2950
-	0    1    1    0
-$EndComp
-Wire Wire Line
-	9000 2600 9000 2800
-$Comp
-L C_Small C4
-U 1 1 58BE5178
-P 9100 2700
-F 0 "C4" V 9150 2750 50  0000 L CNN
-F 1 "0.1uF" V 9050 2750 50  0000 L CNN
-F 2 "Capacitors_SMD:C_0805" H 9100 2700 50  0001 C CNN
-F 3 "" H 9100 2700 50  0000 C CNN
-	1    9100 2700
-	0    1    1    0
-$EndComp
-Wire Wire Line
-	9000 3100 9000 3400
-Connection ~ 9000 2700
-Text GLabel 9350 2700 3    60   Input ~ 0
-GND
-Wire Wire Line
-	9200 2700 9350 2700
 $Comp
 L CONN_01X01 P8
@@
 Text GLabel 6150 1600 2    60   Input ~ 0
 HVGND
-Connection ~ 9000 2050
-Wire Wire Line
-	9300 2050 9000 2050
 Connection ~ 950  3950
 Connection ~ 2200 3950
@@
 	2450 3850 2450 3950
 Connection ~ 2450 3950
-Wire Wire Line
-	10150 1200 10150 3000
-Wire Wire Line
-	10150 3000 9950 3000
-Wire Wire Line
-	9950 3400 9750 3400
-Connection ~ 9950 2050
 Text Notes 650  4300 0    60   ~ 0
 MOUNTING HOLES
@@
 Text GLabel 6200 4450 2    60   Input ~ 0
 +12V
-Text GLabel 9650 3400 3    60   Input ~ 0
-D+
-Text GLabel 9550 3400 3    60   Input ~ 0
-D-
 $EndSCHEMATC

Commit message: Fix part numbers for P3 and P7
Parts:
- P3, P7: value TFM-125-02-L-DH -> TFM-120-02-L-DH; Mfg_Part_No TFM-125-02-L-DH -> TFM-120-02-L-DH
Changed lines of the file:
@@
 P 3650 4050
 F 0 "P7" H 3850 4180 45  0000 L BNN
-F 1 "TFM-125-02-L-DH" V 4050 2750 45  0000 L BNN
+F 1 "TFM-120-02-L-DH" V 4050 2750 45  0000 L BNN
 F 2 "WheelerLab:TFM-120-02-X-DH" H 3680 4200 20  0001 C CNN
 F 3 "" H 3650 4050 60  0000 C CNN
-F 4 "TFM-125-02-L-DH" H 3650 4050 60  0001 C CNN "Mfg_Part_No"
+F 4 "TFM-120-02-L-DH" H 3650 4050 60  0001 C CNN "Mfg_Part_No"
 	1    3650 4050
 	1    0    0    -1
@@
 P 7400 4050
 F 0 "P3" H 7600 4180 45  0000 L BNN
-F 1 "TFM-125-02-L-DH" V 7800 2850 45  0000 L BNN
+F 1 "TFM-120-02-L-DH" V 7800 2850 45  0000 L BNN
 F 2 "WheelerLab:TFM-120-02-X-DH" H 7430 4200 20  0001 C CNN
 F 3 "" H 7400 4050 60  0000 C CNN
-F 4 "TFM-125-02-L-DH" H 7400 4050 60  0001 C CNN "Mfg_Part_No"
+F 4 "TFM-120-02-L-DH" H 7400 4050 60  0001 C CNN "Mfg_Part_No"
 	1    7400 4050
 	1    0    0    -1
