File: dropbot-front-panel.kicad_pcb (KiCad board)
At the start: 4 copper layers, 108 x 68.8 mm, 29 parts, among them P1 SFM-105-02-L-D-A, P10 Conn_01x02, P13 Conn_01x01, P14 Conn_01x01, P15 Conn_01x01, P2 SFM-125-02-L-D-A, P3 TFM-120-01-L-D-RA, P4 SFM-125-02-L-D-A, P5 TFM-125-01-L-D-RA, P6 SFM-125-02-L-D-A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

Commit message: Fix ERC errors
Connections:
- net +12V_SUPPLY renamed /+12V_SUPPLY
- net CH-X1 renamed /CH-X1
- net CH-X2 renamed /CH-X2
Changed lines of the file:
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@@
   (net 135 "Net-(U2-Pad1)")
   (net 136 "Net-(C1-Pad1)")
-  (net 137 +12V_SUPPLY)
-  (net 138 CH-X2)
-  (net 139 CH-X1)
-  (net 140 "Net-(D1-Pad2)")
-  (net 141 "Net-(R7-Pad2)")
-  (net 142 "Net-(JP4-Pad2)")
-  (net 143 "Net-(JP5-Pad2)")
+  (net 137 "Net-(D1-Pad2)")
+  (net 138 "Net-(R7-Pad2)")
+  (net 139 "Net-(JP4-Pad2)")
+  (net 140 "Net-(JP5-Pad2)")
+  (net 141 /CH-X1)
+  (net 142 /CH-X2)
+  (net 143 /+12V_SUPPLY)
   (net_class Default "This is the default net class."
     (clearance 0.15)
@@
     (uvia_drill 0.1)
     (add_net +3.3V)
-    (add_net CH-X1)
-    (add_net CH-X2)
+    (add_net /+12V_SUPPLY)
+    (add_net /CH-X1)
+    (add_net /CH-X2)
     (add_net CHASIS_GND)
     (add_net CUR_SENSE)
@@
     (uvia_drill 0.1)
     (add_net +12V)
-    (add_net +12V_SUPPLY)
     (add_net HVAC)
     (add_net HVGND)
@@
     (fp_line (start 7.79 4) (end -2.71 4) (layer F.CrtYd) (width 0.05))
     (pad 1 thru_hole rect (at 0 0 270) (size 3 3) (drill 1.52) (layers *.Cu *.Mask)
-      (net 137 +12V_SUPPLY))
+      (net 143 /+12V_SUPPLY))
     (pad 2 thru_hole circle (at 5.08 0 270) (size 3 3) (drill 1.52) (layers *.Cu *.Mask)
       (net 133 CHASIS_GND))
@@
       (net 136 "Net-(C1-Pad1)"))
     (pad 4 smd oval (at 1.905 2.794 90) (size 0.6096 1.4732) (layers F.Cu F.Paste F.Mask)
-      (net 140 "Net-(D1-Pad2)"))
+      (net 137 "Net-(D1-Pad2)"))
     (pad 5 smd oval (at 1.905 -2.794 90) (size 0.6096 1.4732) (layers F.Cu F.Paste F.Mask)
-      (net 137 +12V_SUPPLY))
+      (net 143 /+12V_SUPPLY))
     (pad 6 smd oval (at 0.635 -2.794 90) (size 0.6096 1.4732) (layers F.Cu F.Paste F.Mask)
-      (net 137 +12V_SUPPLY))
+      (net 143 /+12V_SUPPLY))
     (pad 7 smd oval (at -0.635 -2.794 90) (size 0.6096 1.4732) (layers F.Cu F.Paste F.Mask)
-      (net 137 +12V_SUPPLY))
+      (net 143 /+12V_SUPPLY))
     (pad 8 smd oval (at -1.905 -2.794 90) (size 0.6096 1.4732) (layers F.Cu F.Paste F.Mask)
-      (net 137 +12V_SUPPLY))
+      (net 143 /+12V_SUPPLY))
   )
   (module Resistors_SMD:R_0805 (layer F.Cu)
@@
       (net 136 "Net-(C1-Pad1)"))
     (pad 2 smd rect (at 1.05 0 180) (size 0.6 0.45) (layers F.Cu F.Paste F.Mask)
-      (net 140 "Net-(D1-Pad2)"))
+      (net 137 "Net-(D1-Pad2)"))
     (model ${KISYS3DMOD}/Diodes_SMD.3dshapes/D_SOD-323.wrl
       (at (xyz 0 0 0))
@@
     (fp_line (start 1.55 0.9) (end -1.55 0.9) (layer F.CrtYd) (width 0.05))
     (pad 1 smd rect (at -0.95 0 180) (size 0.7 1.3) (layers F.Cu F.Paste F.Mask)
-      (net 140 "Net-(D1-Pad2)"))
+      (net 137 "Net-(D1-Pad2)"))
     (pad 2 smd rect (at 0.95 0 180) (size 0.7 1.3) (layers F.Cu F.Paste F.Mask)
       (net 133 CHASIS_GND))
@@
       (net 5 +3.3V))
     (pad 2 smd rect (at 0.95 0 270) (size 0.7 1.3) (layers F.Cu F.Paste F.Mask)
-      (net 141 "Net-(R7-Pad2)"))
+      (net 138 "Net-(R7-Pad2)"))
     (model ${KISYS3DMOD}/Resistors_SMD.3dshapes/R_0805.wrl
       (at (xyz 0 0 0))
@@
       (net 5 +3.3V))
     (pad 2 smd rect (at -2.95 -0.325 90) (size 1.45 0.45) (layers F.Cu F.Paste F.Mask)
-      (net 142 "Net-(JP4-Pad2)"))
+      (net 139 "Net-(JP4-Pad2)"))
     (pad 3 smd rect (at -2.95 0.325 90) (size 1.45 0.45) (layers F.Cu F.Paste F.Mask)
-      (net 143 "Net-(JP5-Pad2)"))
+      (net 140 "Net-(JP5-Pad2)"))
     (pad 4 smd rect (at -2.95 0.975 90) (size 1.45 0.45) (layers F.Cu F.Paste F.Mask)
       (net 2 GND))
@@
       (net 1 SCL))
     (pad 7 smd rect (at 2.95 -0.325 90) (size 1.45 0.45) (layers F.Cu F.Paste F.Mask)
-      (net 141 "Net-(R7-Pad2)"))
+      (net 138 "Net-(R7-Pad2)"))
     (pad 8 smd rect (at 2.95 -0.975 90) (size 1.45 0.45) (layers F.Cu F.Paste F.Mask)
       (net 5 +3.3V))
@@
       (net 5 +3.3V))
     (pad 2 smd rect (at 0.75 0 90) (size 0.5 0.9) (layers F.Cu F.Paste F.Mask)
-      (net 142 "Net-(JP4-Pad2)"))
+      (net 139 "Net-(JP4-Pad2)"))
     (model ${KISYS3DMOD}/Resistors_SMD.3dshapes/R_0603.wrl
       (at (xyz 0 0 0))
@@
       (net 5 +3.3V))
     (pad 2 smd rect (at 0.75 0 90) (size 0.5 0.9) (layers F.Cu F.Paste F.Mask)
-      (net 143 "Net-(JP5-Pad2)"))
+      (net 140 "Net-(JP5-Pad2)"))
     (model ${KISYS3DMOD}/Resistors_SMD.3dshapes/R_0603.wrl
       (at (xyz 0 0 0))
@@
       (net 3 +12V))
     (pad 2 thru_hole circle (at 15.24 7.368) (size 0.814 0.814) (drill 0.56) (layers *.Cu *.Mask F.SilkS)
-      (net 139 CH-X1))
+      (net 141 /CH-X1))
     (pad 1 thru_hole circle (at 15.24 6.098) (size 0.814 0.814) (drill 0.56) (layers *.Cu *.Mask F.SilkS)
-      (net 138 CH-X2))
+      (net 142 /CH-X2))
     (pad 11 thru_hole circle (at 8.89 6.098) (size 0.814 0.814) (drill 0.56) (layers *.Cu *.Mask F.SilkS)
       (net 58 HVOUT79))
@@
   (segment (start 48.3 66) (end 48.8 65.5) (width 0.5) (layer F.Cu) (net 136) (status 30))
   (segment (start 48.1 66.35) (end 48.3 66.15) (width 0.5) (layer F.Cu) (net 136) (status 30))
-  (segment (start 58 48) (end 58.7 48) (width 0.5) (layer F.Cu) (net 137))
-  (segment (start 58.7 48) (end 61.4 50.7) (width 0.5) (layer F.Cu) (net 137))
-  (segment (start 62.501 50.7) (end 63.006 50.195) (width 0.5) (layer F.Cu) (net 137))
-  (segment (start 61.4 50.7) (end 62.501 50.7) (width 0.5) (layer F.Cu) (net 137))
-  (segment (start 63.006 54.005) (end 62.905 54.005) (width 0.5) (layer F.Cu) (net 137))
-  (segment (start 62.905 54.005) (end 62.5 53.6) (width 0.5) (layer F.Cu) (net 137))
-  (segment (start 62.5 50.701) (end 63.006 50.195) (width 0.5) (layer F.Cu) (net 137))
-  (segment (start 62.5 53.6) (end 62.5 50.701) (width 0.5) (layer F.Cu) (net 137))
-  (segment (start 58 48) (end 59.4 48) (width 0.5) (layer F.Cu) (net 137))
-  (segment (start 59.4 48) (end 61.595 50.195) (width 0.5) (layer F.Cu) (net 137))
-  (segment (start 61.595 50.195) (end 63.006 50.195) (width 0.5) (layer F.Cu) (net 137))
-  (segment (start 63.006 52.735) (end 63.006 54.005) (width 0.5) (layer F.Cu) (net 137))
-  (segment (start 63.006 51.465) (end 63.006 52.735) (width 0.5) (layer F.Cu) (net 137))
-  (segment (start 63.006 50.195) (end 63.006 51.465) (width 0.5) (layer F.Cu) (net 137))
-  (segment (start 66.05 48.3) (end 66.699 48.3) (width 0.15) (layer F.Cu) (net 140))
-  (segment (start 66.699 48.3) (end 68.594 50.195) (width 0.15) (layer F.Cu) (net 140))
-  (segment (start 64.75 48.3) (end 66.05 48.3) (width 0.15) (layer F.Cu) (net 140))
-  (segment (start 148.5 70.05) (end 150.75 70.05) (width 0.15) (layer F.Cu) (net 141))
-  (segment (start 151.075 69.725) (end 151.075 68.55) (width 0.15) (layer F.Cu) (net 141))
-  (segment (start 150.75 70.05) (end 151.075 69.725) (width 0.15) (layer F.Cu) (net 141))
-  (segment (start 151.075 74.45) (end 151.075 75.925) (width 0.15) (layer F.Cu) (net 142))
-  (segment (start 151.075 75.925) (end 151.4 76.25) (width 0.15) (layer F.Cu) (net 142))
-  (segment (start 151.725 74.45) (end 151.725 75.225) (width 0.15) (layer F.Cu) (net 143))
-  (segment (start 151.725 75.225) (end 152.7 76.2) (width 0.15) (layer F.Cu) (net 143))
-  (segment (start 152.7 76.2) (end 152.7 76.25) (width 0.15) (layer F.Cu) (net 143))
+  (segment (start 58 48) (end 58.7 48) (width 0.5) (layer F.Cu) (net 143))
+  (segment (start 58.7 48) (end 61.4 50.7) (width 0.5) (layer F.Cu) (net 143))
+  (segment (start 62.501 50.7) (end 63.006 50.195) (width 0.5) (layer F.Cu) (net 143))
+  (segment (start 61.4 50.7) (end 62.501 50.7) (width 0.5) (layer F.Cu) (net 143))
+  (segment (start 63.006 54.005) (end 62.905 54.005) (width 0.5) (layer F.Cu) (net 143))
+  (segment (start 62.905 54.005) (end 62.5 53.6) (width 0.5) (layer F.Cu) (net 143))
+  (segment (start 62.5 50.701) (end 63.006 50.195) (width 0.5) (layer F.Cu) (net 143))
+  (segment (start 62.5 53.6) (end 62.5 50.701) (width 0.5) (layer F.Cu) (net 143))
+  (segment (start 58 48) (end 59.4 48) (width 0.5) (layer F.Cu) (net 143))
+  (segment (start 59.4 48) (end 61.595 50.195) (width 0.5) (layer F.Cu) (net 143))
+  (segment (start 61.595 50.195) (end 63.006 50.195) (width 0.5) (layer F.Cu) (net 143))
+  (segment (start 63.006 52.735) (end 63.006 54.005) (width 0.5) (layer F.Cu) (net 143))
+  (segment (start 63.006 51.465) (end 63.006 52.735) (width 0.5) (layer F.Cu) (net 143))
+  (segment (start 63.006 50.195) (end 63.006 51.465) (width 0.5) (layer F.Cu) (net 143))
+  (segment (start 66.05 48.3) (end 66.699 48.3) (width 0.15) (layer F.Cu) (net 137))
+  (segment (start 66.699 48.3) (end 68.594 50.195) (width 0.15) (layer F.Cu) (net 137))
+  (segment (start 64.75 48.3) (end 66.05 48.3) (width 0.15) (layer F.Cu) (net 137))
+  (segment (start 148.5 70.05) (end 150.75 70.05) (width 0.15) (layer F.Cu) (net 138))
+  (segment (start 151.075 69.725) (end 151.075 68.55) (width 0.15) (layer F.Cu) (net 138))
+  (segment (start 150.75 70.05) (end 151.075 69.725) (width 0.15) (layer F.Cu) (net 138))
+  (segment (start 151.075 74.45) (end 151.075 75.925) (width 0.15) (layer F.Cu) (net 139))
+  (segment (start 151.075 75.925) (end 151.4 76.25) (width 0.15) (layer F.Cu) (net 139))
+  (segment (start 151.725 74.45) (end 151.725 75.225) (width 0.15) (layer F.Cu) (net 140))
+  (segment (start 151.725 75.225) (end 152.7 76.2) (width 0.15) (layer F.Cu) (net 140))
+  (segment (start 152.7 76.2) (end 152.7 76.25) (width 0.15) (layer F.Cu) (net 140))
   (zone (net 2) (net_name GND) (layer F.Cu) (hatch edge 0.508)
     (connect_pads (clearance 0.6))
