File: dropbot-front-panel.sch (KiCad schematic (older format))
At the start: 21 parts, among them P1 SFM-105-02-L-D-A, P10 CONN_01X02, P13 CONN_01X01, P14 CONN_01X01, P15 CONN_01X01, P2 SFM-125-02-L-D-A, P3 TFM-120-02-L-DH, P4 SFM-125-02-L-D-A, P5 TFM-125-02-L-DH, P6 SFM-125-02-L-D-A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

Commit message: Fix #1, #2 and #3
1. Add i2c EEPROM chip to store serial number, hardware version, etc.
2. Move C2 and C3 (they currently collide with the 2nd switching board)
3. Fix reverse polarity protection
Parts:
- added C4: 0.1uF, Capacitors_SMD:C_0805, symbol C_Small
- added D1: 10V, Diodes_SMD:D_SOD-323, symbol D_Zener_Small
- added JP3: A0, Resistors_SMD:R_0603, symbol Jumper_NO_Small
- added JP4: A1, Resistors_SMD:R_0603, symbol Jumper_NO_Small
- added JP5: A2, Resistors_SMD:R_0603, symbol Jumper_NO_Small
- added R1, R7: 10k, Resistors_SMD:R_0805, symbol R_Small
- added U1: CAT24C__, Housings_SSOP:TSSOP-8_4.4x3mm_Pitch0.65mm, symbol CAT24C__
- JP1, JP2: symbol JUMPER -> Jumper
Connections:
- wire segments 28 -> 38
Other:
- note added: "EEPROM"
- moved on the sheet: C1, C2, C3, L2, Q1

Commit message: Update to use Sci-Bots library
Parts:
- removed P1: SFM-105-02-L-D-A, WheelerLab:SFM-105-02-XXX-D-A, symbol CONN_02X05
- removed P10: CONN_01X02, Connect:bornier2, symbol CONN_01X02
- removed P13, P14, P15, P8: CONN_01X01, Connect:1pin, symbol CONN_01X01
- removed P2, P4, P6: SFM-125-02-L-D-A, WheelerLab:SFM-125-02-XXX-D-A, symbol CONN_02X25
- removed P9: CONN_01X03, Pin_Headers:Pin_Header_Straight_1x03, symbol CONN_01X03
- added P1: SFM-105-02-L-D-A, Sci-Bots:SFM-105-02-XXX-D-A, symbol Conn_02x05_Odd_Even
- added P10: Conn_01x02, Connect:bornier2, symbol Conn_01x02
- added P13, P14, P15, P8: Conn_01x01, Connect:1pin, symbol Conn_01x01
- added P2, P4, P6: SFM-125-02-L-D-A, Sci-Bots:SFM-125-02-XXX-D-A, symbol Conn_02x25_Odd_Even
- added P9: Conn_01x03, Pin_Headers:Pin_Header_Straight_1x03, symbol Conn_01x03
- L2: footprint WheelerLab:RN242-X-02-XXX -> Sci-Bots:RN242-X-02-XXX
- P3, P7: footprint WheelerLab:TFM-120-02-X-DH -> Sci-Bots:TFM-120-02-X-DH
- P5: footprint WheelerLab:TFM-125-02-X-DH -> Sci-Bots:TFM-125-02-X-DH
- U2: footprint WheelerLab:D24V22F -> Sci-Bots:D24V22F
Changed lines of the file:
@@
 LIBS:contrib
 LIBS:valves
-LIBS:wheelerlab
+LIBS:sci-bots
+LIBS:dropbot-front-panel-cache
 EELAYER 25 0
 EELAYER END
@@
 Text GLabel 4250 1400 2    60   Input ~ 0
 SCL
-$Comp
-L CONN_02X25 P6
-U 1 1 5847A5CC
-P 4000 2400
-F 0 "P6" H 4000 3700 50  0000 C CNN
-F 1 "SFM-125-02-L-D-A" V 4000 2400 50  0000 C CNN
-F 2 "WheelerLab:SFM-125-02-XXX-D-A" H 4000 1650 50  0001 C CNN
-F 3 "" H 4000 1650 50  0000 C CNN
-F 4 "SFM-125-02-L-D-A" H 4000 2400 60  0001 C CNN "Mfg_Part_No"
-	1    4000 2400
-	1    0    0    -1
-$EndComp
 Text GLabel 3750 1300 0    60   Input ~ 0
 GND
@@
 Text GLabel 5650 3600 0    60   Input ~ 0
 HVOUT41
-$Comp
-L CONN_02X25 P4
-U 1 1 5847BEA4
-P 5900 2400
-F 0 "P4" H 5900 3700 50  0000 C CNN
-F 1 "SFM-125-02-L-D-A" V 5900 2400 50  0000 C CNN
-F 2 "WheelerLab:SFM-125-02-XXX-D-A" H 5900 1650 50  0001 C CNN
-F 3 "" H 5900 1650 50  0000 C CNN
-F 4 "SFM-125-02-L-D-A" H 5900 2400 60  0001 C CNN "Mfg_Part_No"
-	1    5900 2400
-	1    0    0    -1
-$EndComp
 Text GLabel 7500 1900 0    60   Input ~ 0
 HVOUT115
@@
 Text GLabel 7500 3600 0    60   Input ~ 0
 HVOUT81
-$Comp
-L CONN_02X25 P2
-U 1 1 5847C137
-P 7750 2400
-F 0 "P2" H 7750 3700 50  0000 C CNN
-F 1 "SFM-125-02-L-D-A" V 7750 2400 50  0000 C CNN
-F 2 "WheelerLab:SFM-125-02-XXX-D-A" H 7750 1650 50  0001 C CNN
-F 3 "" H 7750 1650 50  0000 C CNN
-F 4 "SFM-125-02-L-D-A" H 7750 2400 60  0001 C CNN "Mfg_Part_No"
-	1    7750 2400
-	1    0    0    -1
-$EndComp
 Text GLabel 5500 4750 0    60   Input ~ 0
 HVOUT75
@@
 Text GLabel 1550 7300 2    60   Input ~ 0
 HV_OE
-$Comp
-L CONN_01X03 P9
-U 1 1 5857AD4F
-P 1150 6250
-F 0 "P9" H 1150 6450 50  0000 C CNN
-F 1 "CONN_01X03" V 1250 6250 50  0001 C CNN
-F 2 "Pin_Headers:Pin_Header_Straight_1x03" H 1150 6250 50  0001 C CNN
-F 3 "" H 1150 6250 50  0000 C CNN
-	1    1150 6250
-	1    0    0    -1
-$EndComp
 Text GLabel 950  6150 0    60   Input ~ 0
 RST1
@@
 F 0 "U2" H 1500 5690 60  0000 C CNN
 F 1 "D24V22F3" H 1500 5205 60  0000 C CNN
-F 2 "WheelerLab:D24V22F" H 1500 5450 60  0001 C CNN
+F 2 "Sci-Bots:D24V22F" H 1500 5450 60  0001 C CNN
 F 3 "" H 1500 5450 60  0000 C CNN
 	1    1500 5450
@@
 Text GLabel 2000 5500 2    60   Input ~ 0
 +3.3V
-$Comp
-L CONN_01X02 P10
-U 1 1 58AE0FFD
-P 1050 3500
-F 0 "P10" H 1050 3650 50  0000 C CNN
-F 1 "CONN_01X02" V 1150 3500 50  0001 C CNN
-F 2 "Connect:bornier2" H 1050 3500 50  0001 C CNN
-F 3 "" H 1050 3500 50  0000 C CNN
-F 4 "ED2609-ND" H 1050 3500 60  0001 C CNN "Mfg_Part_No"
-	1    1050 3500
-	1    0    0    -1
-$EndComp
 Text GLabel 1200 3250 2    60   Input ~ 0
 +12V_SUPPLY
@@
 Text GLabel 2000 5400 2    60   Input ~ 0
 GND
-$Comp
-L CONN_02X05 P1
-U 1 1 58B8600D
-P 1550 1150
-F 0 "P1" H 1550 1450 50  0000 C CNN
-F 1 "SFM-105-02-L-D-A" H 1550 850 50  0000 C CNN
-F 2 "WheelerLab:SFM-105-02-XXX-D-A" H 1550 -50 50  0001 C CNN
-F 3 "" H 1550 -50 50  0000 C CNN
-F 4 "SFM-105-02-L-D-A" H 1550 1150 60  0001 C CNN "Mfg_Part_No"
-	1    1550 1150
-	1    0    0    -1
-$EndComp
 Text GLabel 1800 1250 2    60   Input ~ 0
 +12V
@@
 F 0 "P7" H 3850 4180 45  0000 L BNN
 F 1 "TFM-120-02-L-DH" V 4050 2750 45  0000 L BNN
-F 2 "WheelerLab:TFM-120-02-X-DH" H 3680 4200 20  0001 C CNN
+F 2 "Sci-Bots:TFM-120-02-X-DH" H 3680 4200 20  0001 C CNN
 F 3 "" H 3650 4050 60  0000 C CNN
 F 4 "TFM-120-02-L-DH" H 3650 4050 60  0001 C CNN "Mfg_Part_No"
@@
 F 0 "P3" H 7600 4180 45  0000 L BNN
 F 1 "TFM-120-02-L-DH" V 7800 2850 45  0000 L BNN
-F 2 "WheelerLab:TFM-120-02-X-DH" H 7430 4200 20  0001 C CNN
+F 2 "Sci-Bots:TFM-120-02-X-DH" H 7430 4200 20  0001 C CNN
 F 3 "" H 7400 4050 60  0000 C CNN
 F 4 "TFM-120-02-L-DH" H 7400 4050 60  0001 C CNN "Mfg_Part_No"
@@
 F 0 "P5" H 5700 4180 45  0000 L BNN
 F 1 "TFM-125-02-L-DH" V 5900 2500 45  0000 L BNN
-F 2 "WheelerLab:TFM-125-02-X-DH" H 5530 4200 20  0001 C CNN
+F 2 "Sci-Bots:TFM-125-02-X-DH" H 5530 4200 20  0001 C CNN
 F 3 "" H 5500 4050 60  0000 C CNN
 F 4 "TFM-125-02-L-DH" H 5500 4050 60  0001 C CNN "Mfg_Part_No"
@@
 F 0 "L2" V 2450 3500 50  0000 L CNN
 F 1 "1.8mH" V 2550 3450 50  0000 L CNN
-F 2 "WheelerLab:RN242-X-02-XXX" H 2400 3550 50  0001 C CNN
+F 2 "Sci-Bots:RN242-X-02-XXX" H 2400 3550 50  0001 C CNN
 F 3 "" H 2400 3550 50  0000 C CNN
 F 4 "RN242-6-02-1M8" H 2350 3550 60  0001 C CNN "Mfg_Part_No"
@@
 Text GLabel 2700 3600 2    60   Input ~ 0
 GND
-$Comp
-L CONN_01X01 P8
-U 1 1 58BE68AD
-P 850 4400
-F 0 "P8" H 1000 4400 50  0000 C CNN
-F 1 "CONN_01X01" V 950 4400 50  0001 C CNN
-F 2 "Connect:1pin" H 850 4400 50  0001 C CNN
-F 3 "" H 850 4400 50  0000 C CNN
-	1    850  4400
-	-1   0    0    1
-$EndComp
-$Comp
-L CONN_01X01 P13
-U 1 1 58BE6B3B
-P 850 4500
-F 0 "P13" H 1000 4500 50  0000 C CNN
-F 1 "CONN_01X01" V 950 4500 50  0001 C CNN
-F 2 "Connect:1pin" H 850 4500 50  0001 C CNN
-F 3 "" H 850 4500 50  0000 C CNN
-	1    850  4500
-	-1   0    0    1
-$EndComp
-$Comp
-L CONN_01X01 P14
-U 1 1 58BE6CC3
-P 850 4600
-F 0 "P14" H 1000 4600 50  0000 C CNN
-F 1 "CONN_01X01" V 950 4600 50  0001 C CNN
-F 2 "Connect:1pin" H 850 4600 50  0001 C CNN
-F 3 "" H 850 4600 50  0000 C CNN
-	1    850  4600
-	-1   0    0    1
-$EndComp
-$Comp
-L CONN_01X01 P15
-U 1 1 58BE6CC9
-P 850 4700
-F 0 "P15" H 1000 4700 50  0000 C CNN
-F 1 "CONN_01X01" V 950 4700 50  0001 C CNN
-F 2 "Connect:1pin" H 850 4700 50  0001 C CNN
-F 3 "" H 850 4700 50  0000 C CNN
-	1    850  4700
-	-1   0    0    1
-$EndComp
 Text GLabel 1050 4700 2    60   Input ~ 0
 CHASIS_GND
@@
 Wire Wire Line
 	9200 1000 9000 1000
+$Comp
+L Conn_01x02 P10
+U 1 1 5AA2AFDB
+P 1050 3450
+F 0 "P10" H 1050 3550 50  0000 C CNN
+F 1 "Conn_01x02" H 1050 3250 50  0000 C CNN
+F 2 "Connect:bornier2" H 1050 3450 50  0001 C CNN
+F 3 "" H 1050 3450 50  0001 C CNN
+F 4 "ED2609-ND" H 1050 3450 60  0001 C CNN "Mfg_Part_No"
+	1    1050 3450
+	1    0    0    -1
+$EndComp
+$Comp
+L Conn_01x01 P8
+U 1 1 5AA2BB49
+P 850 4400
+F 0 "P8" H 1000 4400 50  0000 C CNN
+F 1 "Conn_01x01" H 1200 4400 50  0001 C CNN
+F 2 "Connect:1pin" H 850 4400 50  0001 C CNN
+F 3 "" H 850 4400 50  0001 C CNN
+	1    850  4400
+	-1   0    0    1
+$EndComp
+$Comp
+L Conn_01x01 P13
+U 1 1 5AA2BDB3
+P 850 4500
+F 0 "P13" H 1000 4500 50  0000 C CNN
+F 1 "Conn_01x01" H 850 4400 50  0001 C CNN
+F 2 "Connect:1pin" H 850 4500 50  0001 C CNN
+F 3 "" H 850 4500 50  0001 C CNN
+	1    850  4500
+	-1   0    0    1
+$EndComp
+$Comp
+L Conn_01x01 P14
+U 1 1 5AA2BEC2
+P 850 4600
+F 0 "P14" H 1000 4600 50  0000 C CNN
+F 1 "Conn_01x01" H 850 4500 50  0001 C CNN
+F 2 "Connect:1pin" H 850 4600 50  0001 C CNN
+F 3 "" H 850 4600 50  0001 C CNN
+	1    850  4600
+	-1   0    0    1
+$EndComp
+$Comp
+L Conn_01x01 P15
+U 1 1 5AA2BF2D
+P 850 4700
+F 0 "P15" H 1000 4700 50  0000 C CNN
+F 1 "Conn_01x01" H 850 4600 50  0001 C CNN
+F 2 "Connect:1pin" H 850 4700 50  0001 C CNN
+F 3 "" H 850 4700 50  0001 C CNN
+	1    850  4700
+	-1   0    0    1
+$EndComp
+$Comp
+L Conn_01x03 P9
+U 1 1 5AA2CB24
+P 1150 6250
+F 0 "P9" H 1150 6450 50  0000 C CNN
+F 1 "Conn_01x03" H 1150 6050 50  0000 C CNN
+F 2 "Pin_Headers:Pin_Header_Straight_1x03" H 1150 6250 50  0001 C CNN
+F 3 "" H 1150 6250 50  0001 C CNN
+	1    1150 6250
+	1    0    0    -1
+$EndComp
+$Comp
+L Conn_02x05_Odd_Even P1
+U 1 1 5AA2D537
+P 1500 1150
+F 0 "P1" H 1550 1450 50  0000 C CNN
+F 1 "SFM-105-02-L-D-A" H 1550 850 50  0000 C CNN
+F 2 "Sci-Bots:SFM-105-02-XXX-D-A" H 1500 1150 50  0001 C CNN
+F 3 "" H 1500 1150 50  0001 C CNN
+F 4 "SFM-105-02-L-D-A" H 1500 1150 60  0001 C CNN "Mfg_Part_No"
+	1    1500 1150
+	1    0    0    -1
+$EndComp
+$Comp
+L Conn_02x25_Odd_Even P6
+U 1 1 5AA2DAFD
+P 3950 2400
+F 0 "P6" H 4000 3700 50  0000 C CNN
+F 1 "SFM-125-02-L-D-A" V 4000 2400 50  0000 C CNN
+F 2 "Sci-Bots:SFM-125-02-XXX-D-A" H 3950 2400 50  0001 C CNN
+F 3 "" H 3950 2400 50  0001 C CNN
+F 4 "SFM-125-02-L-D-A" H 3950 2400 60  0001 C CNN "Mfg_Part_No"
+	1    3950 2400
+	1    0    0    -1
+$EndComp
+$Comp
+L Conn_02x25_Odd_Even P4
+U 1 1 5AA2E2A4
+P 5850 2400
+F 0 "P4" H 5900 3700 50  0000 C CNN
+F 1 "SFM-125-02-L-D-A" V 5900 2400 50  0000 C CNN
+F 2 "Sci-Bots:SFM-125-02-XXX-D-A" H 5850 2400 50  0001 C CNN
+F 3 "" H 5850 2400 50  0001 C CNN
+F 4 "SFM-125-02-L-D-A" H 5850 2400 60  0001 C CNN "Mfg_Part_No"
+	1    5850 2400
+	1    0    0    -1
+$EndComp
+$Comp
+L Conn_02x25_Odd_Even P2
+U 1 1 5AA2E35C
+P 7700 2400
+F 0 "P2" H 7750 3700 50  0000 C CNN
+F 1 "SFM-125-02-L-D-A" V 7750 2400 50  0000 C CNN
+F 2 "Sci-Bots:SFM-125-02-XXX-D-A" H 7700 2400 50  0001 C CNN
+F 3 "" H 7700 2400 50  0001 C CNN
+F 4 "SFM-125-02-L-D-A" H 7700 2400 60  0001 C CNN "Mfg_Part_No"
+	1    7700 2400
+	1    0    0    -1
+$EndComp
 $EndSCHEMATC

Commit message: Use through-hole connectors to pogo-pin board
Parts:
- removed P3, P7: TFM-120-02-L-DH, Sci-Bots:TFM-120-02-X-DH, symbol TFM-120-02-X-DH
- removed P5: TFM-125-02-L-DH, Sci-Bots:TFM-125-02-X-DH, symbol TFM-125-02-X-DH
- added P3, P7: TFM-120-01-L-D-RA, Sci-Bots:TFM-120-01-XXX-D-RA, symbol Conn_02x20_Odd_Even
- added P5: TFM-125-01-L-D-RA, Sci-Bots:TFM-125-01-XXX-D-RA, symbol Conn_02x25_Odd_Even
- P10: Mfg_Part_No ED2609-ND -> (none)
Connections:
- wire segments 38 -> 29

Commit message: Update routing of TFM connectors, replace eeprom part
Fixes #4
Parts:
- U1: Mfg_Part_No CAT24C16YI-GT3 -> M24C02-DRDW8TP/K
Changed lines of the file:
@@
 Sheet 1 1
 Title "DropBot front panel"
-Date "2018-03-09"
-Rev "3.2"
+Date "2018-05-10"
+Rev "3.3"
 Comp "Sci-Bots Inc."
 Comment1 ""
@@
 F 2 "Housings_SSOP:TSSOP-8_4.4x3mm_Pitch0.65mm" H 9490 1145 60  0001 C CNN
 F 3 "" H 9490 1145 60  0000 C CNN
-F 4 "CAT24C16YI-GT3" H 9500 1150 60  0001 C CNN "Mfg_Part_No"
+F 4 "M24C02-DRDW8TP/K" H 9500 1150 60  0001 C CNN "Mfg_Part_No"
 	1    9500 1150
 	1    0    0    -1

Commit message: Update to kicad 5
Parts:
- C1, C2, C3, C4: symbol C_Small -> Device:C_Small
- D1: symbol D_Zener_Small -> Device:D_Zener_Small
- JP1, JP2: symbol Jumper -> Device:Jumper
- JP3, JP4, JP5: symbol Jumper_NO_Small -> Device:Jumper_NO_Small
- L2: symbol CM_CHOKE -> dropbot-front-panel-rescue:CM_CHOKE
- P1: symbol Conn_02x05_Odd_Even -> dropbot-front-panel-rescue:Conn_02x05_Odd_Even
- P10: symbol Conn_01x02 -> dropbot-front-panel-rescue:Conn_01x02
- P13, P14, P15, P8: symbol Conn_01x01 -> dropbot-front-panel-rescue:Conn_01x01
- P2, P4, P5, P6: symbol Conn_02x25_Odd_Even -> dropbot-front-panel-rescue:Conn_02x25_Odd_Even
- P3, P7: symbol Conn_02x20_Odd_Even -> dropbot-front-panel-rescue:Conn_02x20_Odd_Even
- P9: symbol Conn_01x03 -> dropbot-front-panel-rescue:Conn_01x03
- Q1: symbol IRF9388TRPBF -> dropbot-front-panel-rescue:IRF9388TRPBF
- R1, R7: symbol R_Small -> Device:R_Small
- U1: symbol CAT24C__ -> dropbot-front-panel-rescue:CAT24C__
- U2: symbol D24V22F3 -> dropbot-front-panel-rescue:D24V22F3
Changed lines of the file:
@@
-EESchema Schematic File Version 2
-LIBS:dropbot-front-panel-rescue
-LIBS:power
-LIBS:device
-LIBS:transistors
-LIBS:conn
-LIBS:linear
-LIBS:regul
-LIBS:74xx
-LIBS:cmos4000
-LIBS:adc-dac
-LIBS:memory
-LIBS:xilinx
-LIBS:microcontrollers
-LIBS:dsp
-LIBS:microchip
-LIBS:analog_switches
-LIBS:motorola
-LIBS:texas
-LIBS:intel
-LIBS:audio
-LIBS:interface
-LIBS:digital-audio
-LIBS:philips
-LIBS:display
-LIBS:cypress
-LIBS:siliconi
-LIBS:opto
-LIBS:atmel
-LIBS:contrib
-LIBS:valves
-LIBS:sci-bots
-LIBS:dropbot-front-panel-cache
-EELAYER 25 0
+EESchema Schematic File Version 4
+EELAYER 30 0
 EELAYER END
 $Descr USLetter 11000 8500
@@
 HVGND
 $Comp
-L Jumper JP1
+L Device:Jumper JP1
 U 1 1 5857598B
 P 1250 6800
@@
 HVGND
 $Comp
-L Jumper JP2
+L Device:Jumper JP2
 U 1 1 585759FC
 P 1250 7300
@@
 Reset lines for the switching\nboards can be used for\nfirmware flashing.
 $Comp
-L D24V22F3 U2
+L dropbot-front-panel-rescue:D24V22F3 U2
 U 1 1 58AE01C0
 P 1500 5450
@@
 POWER IN\n+12V input with reverse polarity protection and\nEMI filter.
 $Comp
-L IRF9388TRPBF Q1
+L dropbot-front-panel-rescue:IRF9388TRPBF Q1
 U 1 1 58AF05F3
 P 1500 3650
@@
 HVOUT42
 $Comp
-L CM_CHOKE L2
+L dropbot-front-panel-rescue:CM_CHOKE L2
 U 1 1 58BBF946
 P 2350 3550
@@
 $EndComp
 $Comp
-L C_Small C1
+L Device:C_Small C1
 U 1 1 58BC095B
 P 2100 3600
@@
 $EndComp
 $Comp
-L C_Small C2
+L Device:C_Small C2
 U 1 1 58BC0DA1
 P 2450 3800
@@
 $EndComp
 $Comp
-L C_Small C3
+L Device:C_Small C3
 U 1 1 58BC0DD7
 P 2650 3800
@@
 +12V
 $Comp
-L R_Small R1
+L Device:R_Small R1
 U 1 1 59B962E7
 P 1900 3900
@@
 $EndComp
 $Comp
-L D_Zener_Small D1
+L Device:D_Zener_Small D1
 U 1 1 59B97699
 P 1900 3550
@@
 $EndComp
 $Comp
-L CAT24C__ U1
+L dropbot-front-panel-rescue:CAT24C__ U1
 U 1 1 59BAE18B
 P 9500 1150
@@
 GND
 $Comp
-L R_Small R7
+L Device:R_Small R7
 U 1 1 59BAF290
 P 9900 1100
@@
 EEPROM
 $Comp
-L Jumper_NO_Small JP3
+L Device:Jumper_NO_Small JP3
 U 1 1 59C10FC7
 P 9100 1000
@@
 $EndComp
 $Comp
-L Jumper_NO_Small JP4
+L Device:Jumper_NO_Small JP4
 U 1 1 59C11542
 P 9100 1100
@@
 $EndComp
 $Comp
-L Jumper_NO_Small JP5
+L Device:Jumper_NO_Small JP5
 U 1 1 59C115B5
 P 9100 1200
@@
 $EndComp
 $Comp
-L C_Small C4
+L Device:C_Small C4
 U 1 1 59C1415F
 P 10200 950
@@
 Wire Wire Line
 	850  3450 850  3250
-Connection ~ 1800 3650
 Connection ~ 1800 3550
 Wire Bus Line
@@
 	6250 6650 8650 6650
 Wire Wire Line
-	1800 3450 2250 3450
+	1800 3450 1900 3450
 Wire Wire Line
 	2250 3450 2250 3500
@@
 	2100 3500 2100 3450
 Wire Wire Line
-	1050 4400 1050 4700
+	1050 4400 1050 4500
 Connection ~ 1050 4500
 Connection ~ 1050 4600
 Wire Wire Line
-	1800 3450 1800 3650
-Wire Wire Line
-	1200 3250 1200 3750
+	1800 3450 1800 3550
+Wire Wire Line
+	1200 3250 1200 3450
 Connection ~ 1200 3550
 Connection ~ 1200 3650
@@
 	850  3250 1200 3250
 Wire Wire Line
-	700  4000 2650 4000
+	700  4000 850  4000
 Wire Wire Line
 	850  3550 850  4000
@@
 	9800 1000 10000 1000
 Wire Wire Line
-	10000 850  10000 1100
-Wire Wire Line
-	9000 850  10200 850
+	10000 850  10000 1000
+Wire Wire Line
+	9000 850  10000 850
 Connection ~ 10000 1000
 Wire Bus Line
@@
 	8750 1550 8750 600
 Wire Wire Line
-	9000 850  9000 1200
+	9000 850  9000 1000
 Connection ~ 9000 1000
 Connection ~ 9000 1100
@@
 	9200 1000 9000 1000
 $Comp
-L Conn_01x02 P10
+L dropbot-front-panel-rescue:Conn_01x02 P10
 U 1 1 5AA2AFDB
 P 1050 3450
@@
 $EndComp
 $Comp
-L Conn_01x01 P8
+L dropbot-front-panel-rescue:Conn_01x01 P8
 U 1 1 5AA2BB49
 P 850 4400
@@
 $EndComp
 $Comp
-L Conn_01x01 P13
+L dropbot-front-panel-rescue:Conn_01x01 P13
 U 1 1 5AA2BDB3
 P 850 4500
@@
 $EndComp
 $Comp
-L Conn_01x01 P14
+L dropbot-front-panel-rescue:Conn_01x01 P14
 U 1 1 5AA2BEC2
 P 850 4600
@@
 $EndComp
 $Comp
-L Conn_01x01 P15
+L dropbot-front-panel-rescue:Conn_01x01 P15
 U 1 1 5AA2BF2D
 P 850 4700
@@
 $EndComp
 $Comp
-L Conn_01x03 P9
+L dropbot-front-panel-rescue:Conn_01x03 P9
 U 1 1 5AA2CB24
 P 1150 6250
@@
 $EndComp
 $Comp
-L Conn_02x05_Odd_Even P1
+L dropbot-front-panel-rescue:Conn_02x05_Odd_Even P1
 U 1 1 5AA2D537
 P 1500 1150
@@
 $EndComp
 $Comp
-L Conn_02x25_Odd_Even P6
+L dropbot-front-panel-rescue:Conn_02x25_Odd_Even P6
 U 1 1 5AA2DAFD
 P 3950 2400
@@
 $EndComp
 $Comp
-L Conn_02x25_Odd_Even P4
+L dropbot-front-panel-rescue:Conn_02x25_Odd_Even P4
 U 1 1 5AA2E2A4
 P 5850 2400
@@
 $EndComp
 $Comp
-L Conn_02x25_Odd_Even P2
+L dropbot-front-panel-rescue:Conn_02x25_Odd_Even P2
 U 1 1 5AA2E35C
 P 7700 2400
@@
 $EndComp
 $Comp
-L Conn_02x20_Odd_Even P7
+L dropbot-front-panel-rescue:Conn_02x20_Odd_Even P7
 U 1 1 5AA2FE34
 P 3950 4950
@@
 $EndComp
 $Comp
-L Conn_02x20_Odd_Even P3
+L dropbot-front-panel-rescue:Conn_02x20_Odd_Even P3
 U 1 1 5AA302A3
 P 7700 4950
@@
 $EndComp
 $Comp
-L Conn_02x25_Odd_Even P5
+L dropbot-front-panel-rescue:Conn_02x25_Odd_Even P5
 U 1 1 5AA30416
 P 5850 5250
@@
 	1    0    0    -1
 $EndComp
+Wire Wire Line
+	1800 3550 1800 3650
+Wire Wire Line
+	2100 3450 2250 3450
+Wire Wire Line
+	1050 4500 1050 4600
+Wire Wire Line
+	1050 4600 1050 4700
+Wire Wire Line
+	1200 3550 1200 3650
+Wire Wire Line
+	1200 3650 1200 3750
+Wire Wire Line
+	1200 3450 1200 3550
+Wire Wire Line
+	850  4000 1900 4000
+Wire Wire Line
+	2450 4000 2650 4000
+Wire Wire Line
+	1900 3450 2100 3450
+Wire Wire Line
+	1900 4000 2100 4000
+Wire Wire Line
+	2100 4000 2250 4000
+Wire Wire Line
+	2250 4000 2450 4000
+Wire Wire Line
+	10000 1000 10000 1100
+Wire Wire Line
+	9000 1000 9000 1100
+Wire Wire Line
+	9000 1100 9000 1200
+Wire Wire Line
+	10000 850  10200 850
 $EndSCHEMATC

Commit message: Fix BOM
Parts:
- C1, C2, C3, C4: MPN (none) -> CL21B104KBCNNNC; Manufacturer (none) -> Samsung; Mfg_Part_No CL21B104KBCNNNC -> (none)
- D1: MPN (none) -> MMSZ5240BS-7-F; Manufacturer (none) -> Diodes Inc.; Mfg_Part_No MMSZ5240BS-7-F -> (none)
- JP1: MPN (none) -> RC0805JR-070RL; Manufacturer (none) -> Yageo; Mfg_Part_No RC0805JR-070RL -> (none)
- JP2, JP3, JP4, JP5, P10, P9: MPN (none) -> DNP; Manufacturer (none) -> DNP
- L2: MPN (none) -> RN242-6-02-1M8; Manufacturer (none) -> Schaffner; Mfg_Part_No RN242-6-02-1M8 -> (none)
- P1: MPN (none) -> SFM-105-02-L-D-A; Manufacturer (none) -> Samtec; Mfg_Part_No SFM-105-02-L-D-A -> (none)
- P13, P14, P15, P8: MPN (none) -> SFM-125-02-L-D-A; Manufacturer (none) -> Samtec
- P2, P4, P6: MPN (none) -> TFM-120-01-L-D-RA; Manufacturer (none) -> Samtec; Mfg_Part_No SFM-125-02-L-D-A -> (none)
- P3, P7: MPN (none) -> TFM-125-01-L-D-RA; Manufacturer (none) -> Samtec; Mfg_Part_No TFM-120-01-L-D-RA -> (none)
- P5: MPN (none) -> DNP; Manufacturer (none) -> DNP; Mfg_Part_No TFM-125-01-L-D-RA -> (none)
- Q1: MPN (none) -> IRF9388TRPBF; Manufacturer (none) -> Infineon; Mfg_Part_No IRF9388TRPBF -> (none)
- R1, R7: MPN (none) -> RC0805FR-0710KL; Manufacturer (none) -> Yageo; Mfg_Part_No RC0805FR-0710KL -> (none)
- U1: MPN (none) -> M24C02-DRDW8TP/K; Manufacturer (none) -> STMicroelectronics; Mfg_Part_No M24C02-DRDW8TP/K -> (none)
- U2: MPN (none) -> D24V22F3; Manufacturer (none) -> Pololu
