File: dropbot-front-panel.sch (KiCad schematic (older format))
At the start: 29 parts, among them P1 SFM-105-02-L-D-A, P10 Conn_01x02, P13 Conn_01x01, P14 Conn_01x01, P15 Conn_01x01, P2 SFM-125-02-L-D-A, P3 TFM-120-01-L-D-RA, P4 SFM-125-02-L-D-A, P5 TFM-125-01-L-D-RA, P6 SFM-125-02-L-D-A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

Commit message: Fix ERC errors
Parts:
- L2: symbol dropbot-front-panel-rescue:CM_CHOKE -> sci-bots:CM_CHOKE
- P1: symbol dropbot-front-panel-rescue:Conn_02x05_Odd_Even -> Connector_Generic:Conn_02x05_Odd_Even
- P10: symbol dropbot-front-panel-rescue:Conn_01x02 -> Connector_Generic:Conn_01x02
- P13, P14, P15, P8: symbol dropbot-front-panel-rescue:Conn_01x01 -> Connector_Generic:Conn_01x01
- P2, P4, P5, P6: symbol dropbot-front-panel-rescue:Conn_02x25_Odd_Even -> Connector_Generic:Conn_02x25_Odd_Even
- P3, P7: symbol dropbot-front-panel-rescue:Conn_02x20_Odd_Even -> Connector_Generic:Conn_02x20_Odd_Even
- P9: symbol dropbot-front-panel-rescue:Conn_01x03 -> Connector_Generic:Conn_01x03
- Q1: symbol dropbot-front-panel-rescue:IRF9388TRPBF -> sci-bots:IRF9388TRPBF
- U1: symbol dropbot-front-panel-rescue:CAT24C__ -> sci-bots:CAT24C__
- U2: symbol dropbot-front-panel-rescue:D24V22F3 -> sci-bots:D24V22F3
Connections:
- no-connect marks 2 -> 4
Changed lines of the file:
@@
 $EndComp
 $Comp
-L dropbot-front-panel-rescue:D24V22F3 U2
+L sci-bots:D24V22F3 U2
 U 1 1 58AE01C0
 P 1500 5450
@@
 $EndComp
 $Comp
-L dropbot-front-panel-rescue:IRF9388TRPBF Q1
+L sci-bots:IRF9388TRPBF Q1
 U 1 1 58AF05F3
 P 1500 3650
@@
 $EndComp
 $Comp
-L dropbot-front-panel-rescue:CM_CHOKE L2
+L sci-bots:CM_CHOKE L2
 U 1 1 58BBF946
 P 2350 3550
@@
 $EndComp
 $Comp
-L dropbot-front-panel-rescue:CAT24C__ U1
+L sci-bots:CAT24C__ U1
 U 1 1 59BAE18B
 P 9500 1150
@@
 $EndComp
 $Comp
-L dropbot-front-panel-rescue:Conn_01x02 P10
+L Connector_Generic:Conn_01x02 P10
 U 1 1 5AA2AFDB
 P 1050 3450
@@
 $EndComp
 $Comp
-L dropbot-front-panel-rescue:Conn_01x01 P8
+L Connector_Generic:Conn_01x01 P8
 U 1 1 5AA2BB49
 P 850 4400
@@
 $EndComp
 $Comp
-L dropbot-front-panel-rescue:Conn_01x01 P13
+L Connector_Generic:Conn_01x01 P13
 U 1 1 5AA2BDB3
 P 850 4500
@@
 $EndComp
 $Comp
-L dropbot-front-panel-rescue:Conn_01x01 P14
+L Connector_Generic:Conn_01x01 P14
 U 1 1 5AA2BEC2
 P 850 4600
@@
 $EndComp
 $Comp
-L dropbot-front-panel-rescue:Conn_01x01 P15
+L Connector_Generic:Conn_01x01 P15
 U 1 1 5AA2BF2D
 P 850 4700
@@
 $EndComp
 $Comp
-L dropbot-front-panel-rescue:Conn_01x03 P9
+L Connector_Generic:Conn_01x03 P9
 U 1 1 5AA2CB24
 P 1150 6250
@@
 $EndComp
 $Comp
-L dropbot-front-panel-rescue:Conn_02x05_Odd_Even P1
+L Connector_Generic:Conn_02x05_Odd_Even P1
 U 1 1 5AA2D537
 P 1500 1150
@@
 $EndComp
 $Comp
-L dropbot-front-panel-rescue:Conn_02x25_Odd_Even P6
+L Connector_Generic:Conn_02x25_Odd_Even P6
 U 1 1 5AA2DAFD
 P 3950 2400
@@
 $EndComp
 $Comp
-L dropbot-front-panel-rescue:Conn_02x25_Odd_Even P4
+L Connector_Generic:Conn_02x25_Odd_Even P4
 U 1 1 5AA2E2A4
 P 5850 2400
@@
 $EndComp
 $Comp
-L dropbot-front-panel-rescue:Conn_02x25_Odd_Even P2
+L Connector_Generic:Conn_02x25_Odd_Even P2
 U 1 1 5AA2E35C
 P 7700 2400
@@
 $EndComp
 $Comp
-L dropbot-front-panel-rescue:Conn_02x20_Odd_Even P7
+L Connector_Generic:Conn_02x20_Odd_Even P7
 U 1 1 5AA2FE34
 P 3950 4950
@@
 $EndComp
 $Comp
-L dropbot-front-panel-rescue:Conn_02x20_Odd_Even P3
+L Connector_Generic:Conn_02x20_Odd_Even P3
 U 1 1 5AA302A3
 P 7700 4950
@@
 $EndComp
 $Comp
-L dropbot-front-panel-rescue:Conn_02x25_Odd_Even P5
+L Connector_Generic:Conn_02x25_Odd_Even P5
 U 1 1 5AA30416
 P 5850 5250
@@
 	1    5850 5250
 	1    0    0    -1
+$EndComp
+$Comp
+L power:PWR_FLAG #FLG0101
+U 1 1 61A02DD3
+P 2350 4350
+F 0 "#FLG0101" H 2350 4425 50 0001 C CNN
+F 1 "PWR_FLAG" V 2350 4478 50 0000 L CNN
+F 2 "" H 2350 4350 50 0001 C CNN
+F 3 "~" H 2350 4350 50 0001 C CNN
+	1    2350 4350
+	0    1    1    0
+$EndComp
+$Comp
+L power:PWR_FLAG #FLG0102
+U 1 1 61A03ACE
+P 2350 4450
+F 0 "#FLG0102" H 2350 4525 50 0001 C CNN
+F 1 "PWR_FLAG" V 2350 4578 50 0000 L CNN
+F 2 "" H 2350 4450 50 0001 C CNN
+F 3 "~" H 2350 4450 50 0001 C CNN
+	1    2350 4450
+	0    1    1    0
+$EndComp
+$Comp
+L power:PWR_FLAG #FLG0103
+U 1 1 61A04D56
+P 2350 4550
+F 0 "#FLG0103" H 2350 4625 50 0001 C CNN
+F 1 "PWR_FLAG" V 2350 4678 50 0000 L CNN
+F 2 "" H 2350 4550 50 0001 C CNN
+F 3 "~" H 2350 4550 50 0001 C CNN
+	1    2350 4550
+	0    1    1    0
 $EndComp
 Text Notes 700  750  0    60   ~ 0
@@
 Text GLabel 2000 5500 2    60   Input ~ 0
 +3.3V
-Text GLabel 1200 3250 2    60   Input ~ 0
-+12V_SUPPLY
 Text Notes 700  5100 0    60   ~ 0
 3.3V POWER REGULATOR
@@
 Text Notes 650  4300 0    60   ~ 0
 MOUNTING HOLES
-Text GLabel 6150 4050 2    60   Input ~ 0
-CH-X1
-Text GLabel 5650 4050 0    60   Input ~ 0
-CH-X2
 Text GLabel 5650 4150 0    60   Input ~ 0
 CUR_SENSE
@@
 Text Notes 8800 750  0    60   ~ 0
 EEPROM
+Text Label 1200 3250 0    60   ~ 0
++12V_SUPPLY
+Text GLabel 2350 4350 0    60   Input ~ 0
++12V
+Text GLabel 2350 4450 0    60   Input ~ 0
++3.3V
+Text GLabel 2350 4550 0    60   Input ~ 0
+GND
+Text Label 6150 4050 0    60   ~ 0
+CH-X1
+Text Label 5650 4050 2    60   ~ 0
+CH-X2
 Wire Bus Line
 	550  2750 3050 2750
@@
 	2100 3500 2100 3450
 Wire Wire Line
+	850  3250 1200 3250
+Wire Wire Line
+	700  4000 850  4000
+Wire Wire Line
+	850  3550 850  4000
+Wire Wire Line
+	2100 4000 2100 3700
+Wire Wire Line
+	2250 4000 2250 3600
+Wire Wire Line
+	1800 3800 1900 3800
+Wire Wire Line
+	1900 3800 1900 3650
+Wire Wire Line
+	2450 3500 2650 3500
+Wire Wire Line
+	2450 3600 2700 3600
+Wire Wire Line
+	2650 3500 2650 3700
+Wire Wire Line
+	2650 4000 2650 3900
+Wire Wire Line
+	2450 3700 2450 3600
+Wire Wire Line
+	2450 3900 2450 4000
+Wire Wire Line
+	9800 1000 10000 1000
+Wire Wire Line
+	10000 850  10000 1000
+Wire Wire Line
+	9000 850  10000 850
+Wire Bus Line
+	8750 600  10450 600
+Wire Bus Line
+	10450 600  10450 1550
+Wire Bus Line
+	10450 1550 8750 1550
+Wire Bus Line
+	8750 1550 8750 600
+Wire Wire Line
+	9000 850  9000 1000
+Wire Wire Line
+	10200 850  10200 750
+Wire Wire Line
+	10200 1050 10200 1500
+Wire Wire Line
+	10200 1500 9200 1500
+Wire Wire Line
+	9200 1500 9200 1300
+Wire Wire Line
+	9200 1000 9000 1000
+Wire Wire Line
+	2100 3450 2250 3450
+Wire Wire Line
+	850  4000 1900 4000
+Wire Wire Line
+	2450 4000 2650 4000
+Wire Wire Line
+	1900 3450 2100 3450
+Wire Wire Line
+	1900 4000 2100 4000
+Wire Wire Line
+	2100 4000 2250 4000
+Wire Wire Line
+	2250 4000 2450 4000
+Wire Wire Line
+	10000 1000 10000 1100
+Wire Wire Line
+	9000 1000 9000 1100
+Wire Wire Line
+	9000 1100 9000 1200
+Wire Wire Line
+	10000 850  10200 850
+Wire Wire Line
+	1800 3450 1800 3550
+Wire Wire Line
 	1050 4400 1050 4500
 Wire Wire Line
-	1800 3450 1800 3550
-Wire Wire Line
 	1200 3250 1200 3450
 Wire Wire Line
-	850  3250 1200 3250
-Wire Wire Line
-	700  4000 850  4000
-Wire Wire Line
-	850  3550 850  4000
-Wire Wire Line
-	2100 4000 2100 3700
-Wire Wire Line
-	2250 4000 2250 3600
-Wire Wire Line
-	1800 3800 1900 3800
-Wire Wire Line
-	1900 3800 1900 3650
-Wire Wire Line
-	2450 3500 2650 3500
-Wire Wire Line
-	2450 3600 2700 3600
-Wire Wire Line
-	2650 3500 2650 3700
-Wire Wire Line
-	2650 4000 2650 3900
-Wire Wire Line
-	2450 3700 2450 3600
-Wire Wire Line
-	2450 3900 2450 4000
-Wire Wire Line
-	9800 1000 10000 1000
-Wire Wire Line
-	10000 850  10000 1000
-Wire Wire Line
-	9000 850  10000 850
-Wire Bus Line
-	8750 600  10450 600
-Wire Bus Line
-	10450 600  10450 1550
-Wire Bus Line
-	10450 1550 8750 1550
-Wire Bus Line
-	8750 1550 8750 600
-Wire Wire Line
-	9000 850  9000 1000
-Wire Wire Line
-	10200 850  10200 750
-Wire Wire Line
-	10200 1050 10200 1500
-Wire Wire Line
-	10200 1500 9200 1500
-Wire Wire Line
-	9200 1500 9200 1300
-Wire Wire Line
-	9200 1000 9000 1000
+	1050 4500 1050 4600
+Wire Wire Line
+	1050 4600 1050 4700
+Wire Wire Line
+	1200 3450 1200 3550
+Wire Wire Line
+	1200 3550 1200 3650
+Wire Wire Line
+	1200 3650 1200 3750
 Wire Wire Line
 	1800 3550 1800 3650
-Wire Wire Line
-	2100 3450 2250 3450
-Wire Wire Line
-	1050 4500 1050 4600
-Wire Wire Line
-	1050 4600 1050 4700
-Wire Wire Line
-	1200 3550 1200 3650
-Wire Wire Line
-	1200 3650 1200 3750
-Wire Wire Line
-	1200 3450 1200 3550
-Wire Wire Line
-	850  4000 1900 4000
-Wire Wire Line
-	2450 4000 2650 4000
-Wire Wire Line
-	1900 3450 2100 3450
-Wire Wire Line
-	1900 4000 2100 4000
-Wire Wire Line
-	2100 4000 2250 4000
-Wire Wire Line
-	2250 4000 2450 4000
-Wire Wire Line
-	10000 1000 10000 1100
-Wire Wire Line
-	9000 1000 9000 1100
-Wire Wire Line
-	9000 1100 9000 1200
-Wire Wire Line
-	10000 850  10200 850
-Connection ~ 1800 3550
 Connection ~ 2100 3450
-Connection ~ 1050 4500
-Connection ~ 1050 4600
-Connection ~ 1200 3550
-Connection ~ 1200 3650
-Connection ~ 1200 3450
 Connection ~ 850  4000
 Connection ~ 2450 4000
@@
 Connection ~ 9000 1100
 Connection ~ 10000 850
+Connection ~ 1050 4500
+Connection ~ 1050 4600
+Connection ~ 1200 3450
+Connection ~ 1200 3550
+Connection ~ 1200 3650
+Connection ~ 1800 3550
 NoConn ~ 1000 5300
 NoConn ~ 1000 5400
+NoConn ~ 5650 4050
+NoConn ~ 6150 4050
 $EndSCHEMATC
